File: Power_Supply/powersupply_version_1/_autosave-powersupply_version_1.sch (KiCad schematic (older format))
At the start: 42 parts

Commit message: pwr supply changes
Parts:
- removed C?: 2.5 nF, symbol Device:C_Small
- removed C? (x3): C_Small, symbol Device:C_Small
- removed C? (x2): .1 uF, symbol Device:C_Small
- removed C?: 100nF, symbol Device:C_Small
- removed C? (x6): 1 uF, symbol Device:C_Small
- removed C?: .8 uF, symbol Device:C_Small
- removed C? (x2): 12pF, symbol Device:C_Small
- removed D?: D_Zener, symbol Device:D_Zener_Small
- removed D?: D_Zener_Small, symbol Device:D_Zener_Small
- removed L?: 1 mH, symbol Device:L_Small
- removed M? (x2): MNMOS, symbol pspice:MNMOS
- removed R?: 18.3k, symbol Device:R_Small_US
- removed R?: R_Small_US, symbol Device:R_Small_US
- removed R?: 29.4k, symbol Device:R_Small_US
- removed R?: 1M, symbol Device:R_Small_US
- removed R?: 75k, symbol Device:R_Small_US
- removed R?: 10k, symbol Device:R_Small_US
- removed R?: 200m, symbol Device:R_Small_US
- removed R?: R_Small, symbol Device:R_Small_US
- removed R?: 1k, symbol Device:R_Small_US
- removed R?: 5.13k, symbol Device:R_Small_US
- removed RV?: R_POT_US, symbol Device:R_POT_US
- removed U?: LM25118, symbol powersupply_version_1:LM25118
- removed U?: Atmega328P-AU, symbol powersupply_version_1:Atmega328P-AU
- removed Y?: Crystal, symbol Device:Crystal_Small
- added C? (x2): 0.1uF, symbol Device:C_Small
- added C? (x2): 12pF, symbol Device:C_Small
- added U?: ATSAMD10D14A-SS, Package_SO:SOIC-20W_7.5x12.8mm_P1.27mm, symbol MCU_Microchip_SAMD:ATSAMD10D14A-SS
- added U?: AP1117-15, Package_TO_SOT_SMD:SOT-223-3_TabPin2, symbol Regulator_Linear:AP1117-15
- added Y?: 16MHz, symbol Device:Crystal_Small
Connections:
- net labels added: +3.3V, GNDREF, SS, VREF1
- wire segments 115 -> 25
- no-connect marks 14 -> 11
Other:
- moved on the sheet: J?, R?, SW?, U?
