File: Power_Supply/powersupply_version_1/powersupply_version_1 2.sch (KiCad schematic (older format))
At the start: 38 parts

Commit message: small changes
Connections:
- net +5V: now also U?.5 (V+), U?.5 (V+)
- net GND: now also U?.4 (V-), U?.4 (V-)
- net mayhavetogroundthese: now reaches U?.8 (In2+)
Changed lines of the file:
@@
 EESchema Schematic File Version 4
+LIBS:powersupply_version_1 2-cache
 EELAYER 29 0
 EELAYER END
@@
 	8050 3600 7950 3600
 Wire Wire Line
-	7950 3600 7950 3950
-Wire Wire Line
 	7600 5350 7500 5350
 Wire Wire Line
 	7500 5350 7500 3950
-Wire Wire Line
-	7500 3950 7950 3950
 Connection ~ 7600 5350
 Wire Wire Line
@@
 Wire Wire Line
 	9200 3450 9400 3450
+$Comp
+L power:+5V #PWR?
+U 1 1 5D45F821
+P 8750 4450
+F 0 "#PWR?" H 8750 4300 50  0001 C CNN
+F 1 "+5V" H 8765 4623 50  0000 C CNN
+F 2 "" H 8750 4450 50  0001 C CNN
+F 3 "" H 8750 4450 50  0001 C CNN
+	1    8750 4450
+	1    0    0    -1
+$EndComp
+$Comp
+L power:GND #PWR?
+U 1 1 5D460F2D
+P 8000 4900
+F 0 "#PWR?" H 8000 4650 50  0001 C CNN
+F 1 "GND" H 8005 4727 50  0000 C CNN
+F 2 "" H 8000 4900 50  0001 C CNN
+F 3 "" H 8000 4900 50  0001 C CNN
+	1    8000 4900
+	1    0    0    -1
+$EndComp
+Wire Wire Line
+	8000 4900 8050 4900
+Wire Wire Line
+	8700 4450 8750 4450
+Wire Wire Line
+	7500 3950 7950 3950
+Wire Wire Line
+	7950 3600 7950 3950
+$Comp
+L power:GND #PWR?
+U 1 1 5D46746E
+P 8050 3750
+F 0 "#PWR?" H 8050 3500 50  0001 C CNN
+F 1 "GND" H 8055 3577 50  0000 C CNN
+F 2 "" H 8050 3750 50  0001 C CNN
+F 3 "" H 8050 3750 50  0001 C CNN
+	1    8050 3750
+	1    0    0    -1
+$EndComp
+$Comp
+L power:+5V #PWR?
+U 1 1 5D46A949
+P 8750 3300
+F 0 "#PWR?" H 8750 3150 50  0001 C CNN
+F 1 "+5V" H 8765 3473 50  0000 C CNN
+F 2 "" H 8750 3300 50  0001 C CNN
+F 3 "" H 8750 3300 50  0001 C CNN
+	1    8750 3300
+	1    0    0    -1
+$EndComp
+Wire Wire Line
+	8700 3300 8750 3300
+Text Label 8700 3750 0    50   ~ 0
+mayhavetogroundthese
 $EndSCHEMATC

Commit message: samd10 changes
Parts:
- removed R?: 2.57k, symbol Device:R_Small_US
- removed U?: MCP4706, symbol powersupply_version_1:MCP4706
- added C?: 100nF, symbol Device:C_Small
- added C? (x2): C_Small, symbol Device:C_Small
- added R? (x2): R_Small_US, symbol Device:R_Small_US
- added U?: 1x2Pinheader, symbol powersupply_version_1:1x2Pinheader
Connections:
- net +3V3: now also U?.1 (VCC), U?.17 (VDD), U?.8 (LED)
- net CS: now also U?.13 (PA31/SWDIO)
- net GND: now also C?.2, C?.2
- net MISO: now also U?.9 (PA22)
- net MOSI: now also U?.10 (PA23)
- net SCK: now also U?.8 (PA16); no longer J?.1 (Pin_1)
- net VCC: now also U?.11 (PA28/~RST); no longer U?.1 (VCC), U?.8 (LED)
- net Vlim: now also C?.1, R?.1
- net Vref: now also C?.1, R?.1
- net SWCLK: now reaches U?.12 (PA30/SWCLK)
- net SWCLK: now also J?.1 (Pin_1)
- net at U?.14 (PA24): now also R?.2
- net at U?.15 (PA25): now also R?.2
- net positive_output: now reaches Q?.2 (D), R?.1
- net positive_output: now also C?.1, U?.2
- net negative_output: now reaches R?.1, R?.2
- net negative_output: now also C?.2, U?.1
- no-connect marks 11 -> 10
Other:
- moved on the sheet: C?, J?, R?, RV?, SW?, U?, Y?
