File: Wave_Generator/wavegenerator_verson_1/wavegenerator_v1.sch (KiCad schematic (older format))
At the start: 60 parts, among them J1 01x05, J2 USB_B_Micro, J3 Conn_Coaxial, J4 1x2Pinheader, SW1 button, SW2 button, SW3 SP3T, U1 LinReg, U2 ATmega328P-AU, U3 MC33063AD, U4 MAX038CPP, Y1 16MHz

Commit message: big changes
Parts:
- removed C11: 220pF, Capacitor_THT:C_Rect_L4.0mm_W2.5mm_P2.50mm, symbol Device:C_Small
- added R7: 500, Resistor_THT:R_Axial_DIN0207_L6.3mm_D2.5mm_P10.16mm_Horizontal, symbol Device:R_Small_US
- added R9: 1.42M, Resistor_THT:R_Axial_DIN0207_L6.3mm_D2.5mm_P10.16mm_Horizontal, symbol Device:R_Small_US
- C10: value 15pF -> 470pF
- C9: value 33nF -> 47nF
- R3: value 3.6k -> 4.87k 1%
- R6: value 100 -> 500
- RV1: value 500k -> 1M
- renumbered C12 to C11, R7 to R8
Connections:
- net GND: now also R7.2; no longer R6.2
- net at C11.1, R4.1, RV1.1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: now also R9.2
- net at R3.2, RV1.3: now also R9.1
- net at R8.2, RV3.2: now also R6.2, R7.1
Other:
- moved on the sheet: R1, R2, R6, RV3
Changed lines of the file:
@@
 P 1300 2900
 F 0 "C10" H 1392 2946 50  0000 L CNN
-F 1 "15pF" H 1392 2855 50  0000 L CNN
+F 1 "470pF" H 1392 2855 50  0000 L CNN
 F 2 "Capacitor_THT:C_Rect_L4.0mm_W2.5mm_P2.50mm" H 1300 2900 50  0001 C CNN
 F 3 "~" H 1300 2900 50  0001 C CNN
@@
 P 950 2700
 F 0 "C9" H 1042 2746 50  0000 L CNN
-F 1 "33nF" H 1042 2655 50  0000 L CNN
+F 1 "47nF" H 1042 2655 50  0000 L CNN
 F 2 "Capacitor_THT:C_Rect_L4.0mm_W2.5mm_P2.50mm" H 950 2700 50  0001 C CNN
 F 3 "~" H 950 2700 50  0001 C CNN
@@
 P 2450 1300
 F 0 "R3" V 2250 1250 50  0000 L CNN
-F 1 "3.6k" V 2350 1250 50  0000 L CNN
+F 1 "4.87k 1%" V 2350 1150 50  0000 L CNN
 F 2 "Resistor_THT:R_Axial_DIN0207_L6.3mm_D2.5mm_P10.16mm_Horizontal" H 2450 1300 50  0001 C CNN
 F 3 "~" H 2450 1300 50  0001 C CNN
@@
 U 1 1 5D1D6226
 P 2000 1300
-F 0 "RV1" V 2300 1350 50  0000 R CNN
-F 1 "500k" V 2200 1350 50  0000 R CNN
+F 0 "RV1" V 2200 1300 50  0000 R CNN
+F 1 "1M" V 2100 1250 50  0000 R CNN
 F 2 "wavegenerator_v1:Potentiometer_PTV09A" H 2000 1300 50  0001 C CNN
 F 3 "~" H 2000 1300 50  0001 C CNN
@@
 $EndComp
 $Comp
-L Device:C_Small C12
+L Device:C_Small C11
 U 1 1 5D2356A9
 P 1100 1500
-F 0 "C12" H 1192 1546 50  0000 L CNN
+F 0 "C11" H 1192 1546 50  0000 L CNN
 F 1 "1uF" H 1192 1455 50  0000 L CNN
 F 2 "Capacitor_THT:C_Rect_L4.0mm_W2.5mm_P2.50mm" H 1100 1500 50  0001 C CNN
@@
 	1    0    0    -1
 $EndComp
-Wire Wire Line
-	1950 3050 2650 3050
 $Comp
 L power:GND #PWR029
@@
 $EndComp
 $Comp
-L Device:C_Small C11
-U 1 1 5D573068
-P 1650 2900
-F 0 "C11" H 1742 2946 50  0000 L CNN
-F 1 "220pF" H 1742 2855 50  0000 L CNN
-F 2 "Capacitor_THT:C_Rect_L4.0mm_W2.5mm_P2.50mm" H 1650 2900 50  0001 C CNN
-F 3 "~" H 1650 2900 50  0001 C CNN
-	1    1650 2900
-	1    0    0    -1
-$EndComp
-$Comp
-L power:GND #PWR0101
-U 1 1 5D57D3C7
-P 1650 3050
-F 0 "#PWR0101" H 1650 2800 50  0001 C CNN
-F 1 "GND" H 1655 2877 50  0000 C CNN
-F 2 "" H 1650 3050 50  0001 C CNN
-F 3 "" H 1650 3050 50  0001 C CNN
-	1    1650 3050
-	1    0    0    -1
-$EndComp
-$Comp
 L power:GND #PWR0102
 U 1 1 5D841218
@@
 	1300 2050 950  2050
 Wire Wire Line
-	1650 3000 1650 3050
-Wire Wire Line
-	1650 2800 1300 2800
-Connection ~ 1300 2800
-Wire Wire Line
 	1750 2550 2250 2550
 Wire Wire Line
 	2550 1300 2650 1300
 Wire Wire Line
-	2150 1300 2350 1300
+	2150 1300 2200 1300
 Wire Wire Line
 	1550 1300 1550 1400
 Wire Wire Line
-	1550 1300 1850 1300
+	1550 1300 1750 1300
 Wire Wire Line
 	4050 3200 4050 2950
@@
 Connection ~ 1150 6200
 $Comp
-L Device:R_Small_US R7
+L Device:R_Small_US R8
 U 1 1 5D3AF030
 P 5100 2050
-F 0 "R7" V 5200 2100 50  0000 C CNN
+F 0 "R8" V 5200 2100 50  0000 C CNN
 F 1 "560" V 5300 2100 50  0000 C CNN
 F 2 "Resistor_THT:R_Axial_DIN0207_L6.3mm_D2.5mm_P10.16mm_Horizontal" H 5100 2050 50  0001 C CNN
@@
 L Device:R_POT RV3
 U 1 1 5D65F834
-P 4550 2050
-F 0 "RV3" H 4700 1850 50  0000 C CNN
-F 1 "1k" H 4700 1950 50  0000 C CNN
-F 2 "wavegenerator_v1:Potentiometer_PTV09A" H 4550 2050 50  0001 C CNN
-F 3 "~" H 4550 2050 50  0001 C CNN
-	1    4550 2050
+P 4350 2050
+F 0 "RV3" H 4200 2000 50  0000 C CNN
+F 1 "1k" H 4200 2100 50  0000 C CNN
+F 2 "wavegenerator_v1:Potentiometer_PTV09A" H 4350 2050 50  0001 C CNN
+F 3 "~" H 4350 2050 50  0001 C CNN
+	1    4350 2050
 	1    0    0    1
 $EndComp
@@
 L Device:R_Small_US R1
 U 1 1 5D46E61E
-P 5300 1300
-F 0 "R1" H 5150 1400 50  0000 L CNN
-F 1 "51" H 5150 1300 50  0000 L CNN
-F 2 "Resistor_THT:R_Axial_DIN0207_L6.3mm_D2.5mm_P10.16mm_Horizontal" H 5300 1300 50  0001 C CNN
-F 3 "~" H 5300 1300 50  0001 C CNN
-	1    5300 1300
+P 4900 1300
+F 0 "R1" H 4750 1400 50  0000 L CNN
+F 1 "51" H 4750 1300 50  0000 L CNN
+F 2 "Resistor_THT:R_Axial_DIN0207_L6.3mm_D2.5mm_P10.16mm_Horizontal" H 4900 1300 50  0001 C CNN
+F 3 "~" H 4900 1300 50  0001 C CNN
+	1    4900 1300
 	-1   0    0    -1
 $EndComp
@@
 L Device:R_Small_US R2
 U 1 1 5D4735CE
-P 5300 1700
-F 0 "R2" H 5150 1750 50  0000 L CNN
-F 1 "51" H 5150 1650 50  0000 L CNN
-F 2 "Resistor_THT:R_Axial_DIN0207_L6.3mm_D2.5mm_P10.16mm_Horizontal" H 5300 1700 50  0001 C CNN
-F 3 "~" H 5300 1700 50  0001 C CNN
-	1    5300 1700
+P 4900 1700
+F 0 "R2" H 4750 1750 50  0000 L CNN
+F 1 "51" H 4750 1650 50  0000 L CNN
+F 2 "Resistor_THT:R_Axial_DIN0207_L6.3mm_D2.5mm_P10.16mm_Horizontal" H 4900 1700 50  0001 C CNN
+F 3 "~" H 4900 1700 50  0001 C CNN
+	1    4900 1700
 	-1   0    0    -1
 $EndComp
@@
 L power:+3.3V #PWR0103
 U 1 1 5D4747AA
-P 5300 1200
-F 0 "#PWR0103" H 5300 1050 50  0001 C CNN
-F 1 "+3.3V" H 5315 1373 50  0000 C CNN
-F 2 "" H 5300 1200 50  0001 C CNN
-F 3 "" H 5300 1200 50  0001 C CNN
-	1    5300 1200
+P 4900 1200
+F 0 "#PWR0103" H 4900 1050 50  0001 C CNN
+F 1 "+3.3V" H 4915 1373 50  0000 C CNN
+F 2 "" H 4900 1200 50  0001 C CNN
+F 3 "" H 4900 1200 50  0001 C CNN
+	1    4900 1200
 	-1   0    0    -1
 $EndComp
@@
 L power:GND #PWR0104
 U 1 1 5D475515
-P 5300 1800
-F 0 "#PWR0104" H 5300 1550 50  0001 C CNN
-F 1 "GND" H 5150 1700 50  0000 C CNN
-F 2 "" H 5300 1800 50  0001 C CNN
-F 3 "" H 5300 1800 50  0001 C CNN
-	1    5300 1800
+P 4900 1800
+F 0 "#PWR0104" H 4900 1550 50  0001 C CNN
+F 1 "GND" H 4750 1700 50  0000 C CNN
+F 2 "" H 4900 1800 50  0001 C CNN
+F 3 "" H 4900 1800 50  0001 C CNN
+	1    4900 1800
 	-1   0    0    -1
 $EndComp
 Text Label 4050 1850 0    50   ~ 0
 output
-Text Label 5300 1500 0    50   ~ 0
+Text Label 4900 1500 0    50   ~ 0
 freq
-Wire Wire Line
-	5300 1400 5300 1500
-Wire Wire Line
-	5300 1600 5300 1500
-Connection ~ 5300 1500
 Wire Wire Line
 	9200 3200 9550 3200
@@
 L Device:R_Small_US R6
 U 1 1 5D4BCD51
-P 4350 2050
-F 0 "R6" H 4150 2100 50  0000 L CNN
-F 1 "100" H 4150 2000 50  0000 L CNN
-F 2 "Resistor_THT:R_Axial_DIN0207_L6.3mm_D2.5mm_P10.16mm_Horizontal" H 4350 2050 50  0001 C CNN
-F 3 "~" H 4350 2050 50  0001 C CNN
-	1    4350 2050
+P 4600 1950
+F 0 "R6" H 4650 2000 50  0000 L CNN
+F 1 "500" H 4650 1900 50  0000 L CNN
+F 2 "Resistor_THT:R_Axial_DIN0207_L6.3mm_D2.5mm_P10.16mm_Horizontal" H 4600 1950 50  0001 C CNN
+F 3 "~" H 4600 1950 50  0001 C CNN
+	1    4600 1950
 	1    0    0    -1
 $EndComp
 Connection ~ 4350 1850
 Wire Wire Line
-	4350 1850 4550 1850
-Wire Wire Line
-	4550 1850 4550 1900
-Wire Wire Line
-	4550 2200 4550 2250
-Wire Wire Line
-	4550 2250 4350 2250
-Wire Wire Line
-	4350 1850 4350 1950
-Wire Wire Line
-	4350 2150 4350 2250
-Connection ~ 4350 2250
-Wire Wire Line
 	4350 1750 4350 1850
 Wire Wire Line
 	4350 1550 4350 1500
-Wire Wire Line
-	4350 1500 5300 1500
-Wire Wire Line
-	4700 2050 5000 2050
 $Comp
 L Device:C_Small C5
@@
 	4650 3400 4650 3600
 Connection ~ 4650 3600
+Wire Wire Line
+	4350 1850 4600 1850
+$Comp
+L Device:R_Small_US R7
+U 1 1 5D440958
+P 4600 2150
+F 0 "R7" H 4668 2196 50  0000 L CNN
+F 1 "500" H 4668 2105 50  0000 L CNN
+F 2 "Resistor_THT:R_Axial_DIN0207_L6.3mm_D2.5mm_P10.16mm_Horizontal" H 4600 2150 50  0001 C CNN
+F 3 "~" H 4600 2150 50  0001 C CNN
+	1    4600 2150
+	1    0    0    -1
+$EndComp
+Wire Wire Line
+	4350 2250 4600 2250
+Wire Wire Line
+	4350 2200 4350 2250
+Connection ~ 4350 2250
+Wire Wire Line
+	4350 1850 4350 1900
+Wire Wire Line
+	4600 2050 5000 2050
+Connection ~ 4600 2050
+Wire Wire Line
+	4500 2050 4600 2050
+Wire Wire Line
+	4900 1400 4900 1500
+Wire Wire Line
+	4350 1500 4900 1500
+Connection ~ 4900 1500
+Wire Wire Line
+	4900 1500 4900 1600
+Wire Wire Line
+	1950 3050 2650 3050
+$Comp
+L Device:R_Small_US R9
+U 1 1 5D422A8A
+P 2000 1000
+F 0 "R9" V 1795 1000 50  0000 C CNN
+F 1 "1.42M" V 1886 1000 50  0000 C CNN
+F 2 "Resistor_THT:R_Axial_DIN0207_L6.3mm_D2.5mm_P10.16mm_Horizontal" H 2000 1000 50  0001 C CNN
+F 3 "~" H 2000 1000 50  0001 C CNN
+	1    2000 1000
+	0    1    1    0
+$EndComp
+Wire Wire Line
+	2100 1000 2200 1000
+Wire Wire Line
+	2200 1000 2200 1300
+Connection ~ 2200 1300
+Wire Wire Line
+	2200 1300 2350 1300
+Wire Wire Line
+	1900 1000 1750 1000
+Wire Wire Line
+	1750 1000 1750 1300
+Connection ~ 1750 1300
+Wire Wire Line
+	1750 1300 1850 1300
 $EndSCHEMATC

Commit message: big changes
Parts:
- renumbered R8 to R10, R9 to R4, R4 to R5, R5 to R6, R7 to R8, R6 to R9
Changed lines of the file:
@@
 $EndComp
 $Comp
-L Device:R_Small_US R4
+L Device:R_Small_US R5
 U 1 1 5D1CCA8A
 P 1550 1600
-F 0 "R4" H 1618 1646 50  0000 L CNN
+F 0 "R5" H 1618 1646 50  0000 L CNN
 F 1 "560" H 1618 1555 50  0000 L CNN
 F 2 "Resistor_THT:R_Axial_DIN0207_L6.3mm_D2.5mm_P10.16mm_Horizontal" H 1550 1600 50  0001 C CNN
@@
 Connection ~ 1850 1300
 $Comp
-L Device:R_Small_US R5
+L Device:R_Small_US R6
 U 1 1 5D1DA50B
 P 1900 1900
-F 0 "R5" H 1968 1946 50  0000 L CNN
+F 0 "R6" H 1968 1946 50  0000 L CNN
 F 1 "180k" H 1968 1855 50  0000 L CNN
 F 2 "Resistor_THT:R_Axial_DIN0207_L6.3mm_D2.5mm_P10.16mm_Horizontal" H 1900 1900 50  0001 C CNN
@@
 Connection ~ 1150 6200
 $Comp
-L Device:R_Small_US R8
+L Device:R_Small_US R10
 U 1 1 5D3AF030
 P 5100 2050
-F 0 "R8" V 5200 2100 50  0000 C CNN
+F 0 "R10" V 5200 2100 50  0000 C CNN
 F 1 "560" V 5300 2100 50  0000 C CNN
 F 2 "Resistor_THT:R_Axial_DIN0207_L6.3mm_D2.5mm_P10.16mm_Horizontal" H 5100 2050 50  0001 C CNN
@@
 	6150 2050 6150 2450
 $Comp
-L Device:R_Small_US R6
+L Device:R_Small_US R9
 U 1 1 5D4BCD51
 P 4600 1950
-F 0 "R6" H 4650 2000 50  0000 L CNN
+F 0 "R9" H 4650 2000 50  0000 L CNN
 F 1 "500" H 4650 1900 50  0000 L CNN
 F 2 "Resistor_THT:R_Axial_DIN0207_L6.3mm_D2.5mm_P10.16mm_Horizontal" H 4600 1950 50  0001 C CNN
@@
 	4350 1850 4600 1850
 $Comp
-L Device:R_Small_US R7
+L Device:R_Small_US R8
 U 1 1 5D440958
 P 4600 2150
-F 0 "R7" H 4668 2196 50  0000 L CNN
+F 0 "R8" H 4668 2196 50  0000 L CNN
 F 1 "500" H 4668 2105 50  0000 L CNN
 F 2 "Resistor_THT:R_Axial_DIN0207_L6.3mm_D2.5mm_P10.16mm_Horizontal" H 4600 2150 50  0001 C CNN
@@
 	1950 3050 2650 3050
 $Comp
-L Device:R_Small_US R9
+L Device:R_Small_US R4
 U 1 1 5D422A8A
 P 2000 1000
-F 0 "R9" V 1795 1000 50  0000 C CNN
+F 0 "R4" V 1795 1000 50  0000 C CNN
 F 1 "1.42M" V 1886 1000 50  0000 C CNN
 F 2 "Resistor_THT:R_Axial_DIN0207_L6.3mm_D2.5mm_P10.16mm_Horizontal" H 2000 1000 50  0001 C CNN
