File: Wave_Generator/wavegenerator_verson_1/wavegenerator_v1.sch (KiCad schematic (older format))
At the start: 61 parts, among them J1 01x05, J2 USB_B_Micro, J3 Conn_Coaxial, J4 1x2Pinheader, SW1 button, SW2 button, SW3 SP3T, U1 LinReg, U2 ATmega328P-AU, U3 MC33063AD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

Commit message: ugh
Parts:
- added R5: 120k, symbol Device:R_Small_US
- R4: value 1.42M -> 1.3M
- renumbered R5 to R6, R6 to R7
Connections:
- net at R3.2, RV1.3: now also R5.1; no longer R4.1
- new net: R4.1, R5.2
Other:
- moved on the sheet: R4
Changed lines of the file:
@@
 $EndComp
 $Comp
-L Device:R_Small_US R5
+L Device:R_Small_US R6
 U 1 1 5D1CCA8A
 P 1550 1600
-F 0 "R5" H 1618 1646 50  0000 L CNN
+F 0 "R6" H 1618 1646 50  0000 L CNN
 F 1 "560" H 1618 1555 50  0000 L CNN
 F 2 "Resistor_THT:R_Axial_DIN0207_L6.3mm_D2.5mm_P10.16mm_Horizontal" H 1550 1600 50  0001 C CNN
@@
 Connection ~ 1850 1300
 $Comp
-L Device:R_Small_US R6
+L Device:R_Small_US R7
 U 1 1 5D1DA50B
 P 1900 1900
-F 0 "R6" H 1968 1946 50  0000 L CNN
+F 0 "R7" H 1968 1946 50  0000 L CNN
 F 1 "180k" H 1968 1855 50  0000 L CNN
 F 2 "Resistor_THT:R_Axial_DIN0207_L6.3mm_D2.5mm_P10.16mm_Horizontal" H 1900 1900 50  0001 C CNN
@@
 Wire Wire Line
 	2550 1300 2650 1300
-Wire Wire Line
-	2150 1300 2200 1300
 Wire Wire Line
 	1550 1300 1550 1400
@@
 L Device:R_Small_US R4
 U 1 1 5D422A8A
-P 2000 1000
-F 0 "R4" V 1795 1000 50  0000 C CNN
-F 1 "1.42M" V 1886 1000 50  0000 C CNN
-F 2 "Resistor_THT:R_Axial_DIN0207_L6.3mm_D2.5mm_P10.16mm_Horizontal" H 2000 1000 50  0001 C CNN
-F 3 "~" H 2000 1000 50  0001 C CNN
-	1    2000 1000
+P 1850 1000
+F 0 "R4" V 1645 1000 50  0000 C CNN
+F 1 "1.3M" V 1736 1000 50  0000 C CNN
+F 2 "Resistor_THT:R_Axial_DIN0207_L6.3mm_D2.5mm_P10.16mm_Horizontal" H 1850 1000 50  0001 C CNN
+F 3 "~" H 1850 1000 50  0001 C CNN
+	1    1850 1000
 	0    1    1    0
 $EndComp
-Wire Wire Line
-	2100 1000 2200 1000
-Wire Wire Line
-	2200 1000 2200 1300
-Connection ~ 2200 1300
-Wire Wire Line
-	2200 1300 2350 1300
-Wire Wire Line
-	1900 1000 1750 1000
 Wire Wire Line
 	1750 1000 1750 1300
@@
 Wire Wire Line
 	1750 1300 1850 1300
+$Comp
+L Device:R_Small_US R5
+U 1 1 5D47F25A
+P 2150 1000
+F 0 "R5" V 1945 1000 50  0000 C CNN
+F 1 "120k" V 2036 1000 50  0000 C CNN
+F 2 "" H 2150 1000 50  0001 C CNN
+F 3 "~" H 2150 1000 50  0001 C CNN
+	1    2150 1000
+	0    1    1    0
+$EndComp
+Wire Wire Line
+	2150 1300 2250 1300
+Wire Wire Line
+	2250 1000 2250 1300
+Connection ~ 2250 1300
+Wire Wire Line
+	2250 1300 2350 1300
+Wire Wire Line
+	1950 1000 2050 1000
 $EndSCHEMATC

Commit message: layout
Parts:
- R5: footprint (none) -> Resistor_THT:R_Axial_DIN0207_L6.3mm_D2.5mm_P10.16mm_Horizontal
- R8, R9: value 500 -> 560
- renumbered C8 to C10, C10 to C8
Connections:
- net at SW3.1: now also C10.1; no longer C8.1
- net at SW3.4: now also C8.1; no longer C10.1
Other:
- moved on the sheet: C10, C8
Changed lines of the file:
@@
 $EndComp
+$Comp
+L Device:C_Small C8
+U 1 1 5D379378
+P 800 2150
+F 0 "C8" H 892 2196 50  0000 L CNN
+F 1 "470pF" H 892 2105 50  0000 L CNN
+F 2 "Capacitor_THT:C_Rect_L4.0mm_W2.5mm_P2.50mm" H 800 2150 50  0001 C CNN
+F 3 "~" H 800 2150 50  0001 C CNN
+	1    800  2150
+	1    0    0    -1
+$EndComp
+Wire Wire Line
+	1300 2650 1300 2800
+Wire Wire Line
+	800  2250 800  2300
+Wire Wire Line
+	950  2550 950  2600
+Wire Wire Line
+	1350 2550 950  2550
+Wire Wire Line
+	1350 2650 1300 2650
 $Comp
 L Device:C_Small C10
-U 1 1 5D379378
+U 1 1 5D37A6B1
 P 1300 2900
 F 0 "C10" H 1392 2946 50  0000 L CNN
-F 1 "470pF" H 1392 2855 50  0000 L CNN
+F 1 "4.7uF" H 1392 2855 50  0000 L CNN
 F 2 "Capacitor_THT:C_Rect_L4.0mm_W2.5mm_P2.50mm" H 1300 2900 50  0001 C CNN
 F 3 "~" H 1300 2900 50  0001 C CNN
 	1    1300 2900
-	1    0    0    -1
-$EndComp
-Wire Wire Line
-	1300 2650 1300 2800
-Wire Wire Line
-	1300 3000 1300 3050
-Wire Wire Line
-	950  2550 950  2600
-Wire Wire Line
-	1350 2550 950  2550
-Wire Wire Line
-	1350 2650 1300 2650
-$Comp
-L Device:C_Small C8
-U 1 1 5D37A6B1
-P 950 2150
-F 0 "C8" H 1042 2196 50  0000 L CNN
-F 1 "4.7uF" H 1042 2105 50  0000 L CNN
-F 2 "Capacitor_THT:C_Rect_L4.0mm_W2.5mm_P2.50mm" H 950 2150 50  0001 C CNN
-F 3 "~" H 950 2150 50  0001 C CNN
-	1    950  2150
 	1    0    0    -1
 $EndComp
@@
 L power:GND #PWR012
 U 1 1 5D3B016C
-P 950 2250
-F 0 "#PWR012" H 950 2000 50  0001 C CNN
-F 1 "GND" H 955 2077 50  0000 C CNN
-F 2 "" H 950 2250 50  0001 C CNN
-F 3 "" H 950 2250 50  0001 C CNN
-	1    950  2250
+P 1300 3000
+F 0 "#PWR012" H 1300 2750 50  0001 C CNN
+F 1 "GND" H 1305 2827 50  0000 C CNN
+F 2 "" H 1300 3000 50  0001 C CNN
+F 3 "" H 1300 3000 50  0001 C CNN
+	1    1300 3000
 	1    0    0    -1
 $EndComp
@@
 L power:GND #PWR016
 U 1 1 5D3BFFC6
-P 1300 3050
-F 0 "#PWR016" H 1300 2800 50  0001 C CNN
-F 1 "GND" H 1305 2877 50  0000 C CNN
-F 2 "" H 1300 3050 50  0001 C CNN
-F 3 "" H 1300 3050 50  0001 C CNN
-	1    1300 3050
+P 800 2300
+F 0 "#PWR016" H 800 2050 50  0001 C CNN
+F 1 "GND" H 805 2127 50  0000 C CNN
+F 2 "" H 800 2300 50  0001 C CNN
+F 3 "" H 800 2300 50  0001 C CNN
+	1    800  2300
 	1    0    0    -1
 $EndComp
@@
 Wire Wire Line
 	1300 2450 1300 2050
-Wire Wire Line
-	1300 2050 950  2050
 Wire Wire Line
 	1750 2550 2250 2550
@@
 P 4600 1950
 F 0 "R9" H 4650 2000 50  0000 L CNN
-F 1 "500" H 4650 1900 50  0000 L CNN
+F 1 "560" H 4650 1900 50  0000 L CNN
 F 2 "Resistor_THT:R_Axial_DIN0207_L6.3mm_D2.5mm_P10.16mm_Horizontal" H 4600 1950 50  0001 C CNN
 F 3 "~" H 4600 1950 50  0001 C CNN
@@
 P 4600 2150
 F 0 "R8" H 4668 2196 50  0000 L CNN
-F 1 "500" H 4668 2105 50  0000 L CNN
+F 1 "560" H 4668 2105 50  0000 L CNN
 F 2 "Resistor_THT:R_Axial_DIN0207_L6.3mm_D2.5mm_P10.16mm_Horizontal" H 4600 2150 50  0001 C CNN
 F 3 "~" H 4600 2150 50  0001 C CNN
@@
 F 0 "R5" V 1945 1000 50  0000 C CNN
 F 1 "120k" V 2036 1000 50  0000 C CNN
-F 2 "" H 2150 1000 50  0001 C CNN
+F 2 "Resistor_THT:R_Axial_DIN0207_L6.3mm_D2.5mm_P10.16mm_Horizontal" H 2150 1000 50  0001 C CNN
 F 3 "~" H 2150 1000 50  0001 C CNN
 	1    2150 1000
@@
 Wire Wire Line
 	1950 1000 2050 1000
+Wire Wire Line
+	800  2050 1300 2050
 $EndSCHEMATC

Commit message: Version 2
Parts:
- removed R5: 120k, Resistor_THT:R_Axial_DIN0207_L6.3mm_D2.5mm_P10.16mm_Horizontal, symbol Device:R_Small_US
- C1, C2: value 100uF -> 220uF 10V; footprint Capacitor_THT:CP_Radial_D6.3mm_P2.50mm -> Capacitor_THT:CP_Radial_D8.0mm_P2.50mm
- C103: value 1500pF -> 560pF
- C106, C107: value 0.1uF -> 1uF
- R1, R2: value 51 -> 182k
- R101: value 0.24 -> 1.5
- R102: value 3.32k -> 3.32k 1%
- R103: value 10k -> 10k 1%
- R4: value 1.3M -> 1.5M 1%
- R5: renamed from R7; value 180k -> 182k 1%
- R6: value 560 -> 549 1%
- R7: renamed from R8; value 560 -> 549
- R8: renamed from R9; value 560 -> 549
- R9: renamed from R10; value 560 -> 549
- TP7: renamed from TP8; value output -> MAX038 Out
- U1: value LinReg -> AZ1117E-3.3
- renumbered TP2 to TP1, TP7 to TP2, TP4 to TP3, TP3 to TP4, TP1 to TP8
Connections:
- net output: now also J3.1 (In), J4.1, R9.1; no longer C3.2, R8.1, RV3.3, TP7.1
- net at R3.2, RV1.3: now also R4.1
- new net MAX038_output: C3.2, R8.1, RV3.3, TP7.1
- no-connect marks 6 -> 16
Other:
- moved on the sheet: C103, C3, H1, H2, H3, H4, R4, R8, TP7
