File: Wave_Generator/wavegenerator_verson_1/wavegenerator_v1.kicad_pcb (KiCad board)
At the start: 2 copper layers, 89.1 x 60 mm, 61 parts, among them J1 01x05, J2 USB_B_Micro, J3 Conn_Coaxial, J4 1x2Pinheader, SW1 button, SW2 button, SW3 SP3T, U1 LinReg, U2 ATmega328P-AU, U3 MC33063AD, U4 MAX038CPP, Y1 16MHz

Commit message: ugh
Parts:
- added R5: 120k, Resistor_THT:R_Axial_DIN0207_L6.3mm_D2.5mm_P10.16mm_Horizontal, F.Cu at (117.9, 44.6)
- R4: value 1.42M -> 1.3M
- moved R4 29.6 mm to (147.4, 55.9), turned to 180 degrees
- moved C11 12.8 mm to (100.5, 62.3)
- moved C8 0.67 mm to (100.6, 49.5)
- moved C9 0.67 mm to (100.6, 53.8)
- moved SW3 0.67 mm to (105.9, 54.4)
- moved C10 0.67 mm to (100.5, 57.9)
- moved R3 0.07 mm to (114.2, 44.6)
- renumbered R5 to R6, R6 to R7
Connections:
- R4 pad 1: Net-(R3-Pad2) -> Net-(R4-Pad1)
Routing:
- net Net-(R3-Pad2): track 11.2 -> 0.00 mm
- net Net-(C11-Pad1): track 85.5 -> 88.1 mm
- net Net-(SW3-Pad2): track 13.6 -> 14.5 mm
- net Net-(R7-Pad2): track 47.4 -> 46.9 mm

Commit message: layout
Parts:
- moved R4 28.6 mm to (119.5, 62.2)
- moved R6 11.1 mm to (103.3, 69.8), turned to 0 degrees
- moved R7 1.93 mm to (103.3, 66.4)
- moved TP5 1.36 mm to (115.6, 78.0)
- moved TP8 0.88 mm to (115.7, 82.5)
Routing:
- net Net-(R3-Pad2): track 0.00 -> 22.9 mm
- net Net-(R7-Pad2): track 46.9 -> 60.1 mm
- net Net-(R4-Pad1): track 0.00 -> 8.17 mm
- net Net-(R6-Pad2): track 26.0 -> 23.9 mm
- net Net-(R10-Pad2): track 52.4 -> 53.4 mm

Commit message: layout
Parts:
- moved R9 15.7 mm to (90.0, 79.1), turned to 0 degrees
- moved R10 9.37 mm to (100.2, 82.5), turned to 180 degrees
- moved C10 8.68 mm to (100.7, 58.2)
- moved R8 8.64 mm to (100.0, 75.7), turned to 180 degrees
- moved C8 8.05 mm to (100.5, 49.9)
- moved R5 6.55 mm to (118.1, 51.1)
- moved R4 6.55 mm to (113.3, 64.4)
- moved R3 6.55 mm to (114.3, 51.1)
- moved C2 6.01 mm to (88.9, 90.4), turned to 90 degrees
- moved C103 4.32 mm to (79.6, 87.6)
- moved D1 3.84 mm to (83.5, 87.2)
- moved R6 2.40 mm to (103.1, 72.2)
- moved R7 2.09 mm to (103.1, 68.5)
- moved L1 1.94 mm to (82.6, 96.6), turned to 0 degrees
- moved R102 1.33 mm to (74.8, 90.4)
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- renumbered C8 to C10, C10 to C8
Connections:
- C10 pad 1: Net-(C8-Pad1) -> Net-(C10-Pad1)
- C8 pad 1: Net-(C10-Pad1) -> Net-(C8-Pad1)
Routing:
- net -5V: track 67.4 -> 54.0 mm
- net Net-(R7-Pad2): track 60.1 -> 48.6 mm
- net /output: track 53.4 -> 63.3 mm
- net Net-(J3-Pad1): track 21.7 -> 29.8 mm
- net Net-(R10-Pad2): track 53.4 -> 46.3 mm
- net Net-(C11-Pad1): track 88.6 -> 95.0 mm
- net Net-(D1-Pad1): track 19.3 -> 14.5 mm
- net Net-(R3-Pad2): track 22.9 -> 18.5 mm
- net +5V: track 161.9 -> 157.6 mm, vias 0 -> 2
- net Net-(C103-Pad1): track 6.88 -> 10.3 mm
- net /WS_0: track 63.2 -> 66.0 mm
- net Net-(R4-Pad1): track 8.17 -> 6.06 mm
- net Net-(R102-Pad1): track 6.46 -> 7.78 mm
- net Net-(R6-Pad2): track 23.9 -> 25.2 mm
- net Net-(R3-Pad1): track 20.5 -> 21.3 mm

Commit message: Version 2
Parts:
- removed the R5 at (118.1, 51.1)
- removed the TP1 at (72.1, 44.8)
- added TP8: GND, TestPoint:TestPoint_THTPad_2.5x2.5mm_Drill1.2mm, F.Cu at (120.9, 45.6)
- C1, C2: footprint Capacitor_THT:CP_Radial_D6.3mm_P2.50mm -> Capacitor_THT:CP_Radial_D8.0mm_P2.50mm
- C103: value 1500pF -> 560pF
- C106, C107: value 0.1uF -> 1uF
- R4: value 1.3M -> 1.5M 1%
- R7: renamed from R8; value 500 -> 560
- R8: renamed from R9; value 500 -> 560
- U1: value LinReg -> AZ1117E-3.3
- moved TP6 51.3 mm to (114.6, 77.6)
- moved TP5 6.39 mm to (109.2, 77.6)
- moved C2 4.64 mm to (93.5, 89.8), turned to 180 degrees
- moved C103 2.91 mm to (81.9, 89.3)
- moved R103 2.91 mm to (73.8, 90.6)
- moved D1 2.75 mm to (85.2, 89.4)
- moved C1 2.75 mm to (67.3, 89.1), turned to 180 degrees
- moved Y1 2.71 mm to (75.5, 84.4)
- moved R3 2.58 mm to (116.4, 49.6)
- moved R102 1.71 mm to (76.5, 90.6)
- moved C105 1.60 mm to (76.2, 80.4)
- moved C104 1.60 mm to (72.3, 80.4)
- moved H1 1.15 mm to (132.1, 45.5)
- moved TP7 1.14 mm to (114.6, 82.9)
- moved H2 1.00 mm to (132.1, 98.5)
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- renumbered R7 to R5, R10 to R9, TP2 to TP1, TP7 to TP2, TP4 to TP3, TP3 to TP4, TP8 to TP7
Connections:
- R4 pad 1: Net-(R4-Pad1) -> Net-(R3-Pad2)
Routing:
- net Net-(R4-Pad1): track 6.06 -> 0.00 mm
- net /WS_0: track 66.0 -> 60.9 mm
- net /WS_1: track 67.1 -> 70.6 mm
- net Net-(R3-Pad1): track 21.3 -> 24.3 mm
- net Net-(C11-Pad1): track 95.0 -> 92.6 mm
- net +5V: track 157.6 -> 159.8 mm, vias 2 -> 1
- net -5V: track 54.0 -> 56.0 mm
- net Net-(D1-Pad1): track 14.5 -> 12.8 mm
- net Net-(C104-Pad2): track 9.37 -> 10.3 mm
- net /switch_n: track 20.4 -> 21.3 mm, vias 1 -> 0
- net /MOSI: track 68.8 -> 68.0 mm
- net Net-(R3-Pad2): track 18.5 -> 17.8 mm
- net Net-(C103-Pad1): track 10.3 -> 9.60 mm
- net /SCK: track 66.1 -> 66.7 mm
- net Net-(R5-Pad2): track 48.6 -> 48.0 mm
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Other:
- board size 89.1 x 60 mm -> 90.1 x 60 mm
- board text added: "Freq"
- board text added: "MAX038 Out"
- board text added: "OUT GND"
- board text added: "WS0"
- board text added: "WS1"
