File: Power_Supply/powersupply/powersupply.sch (KiCad schematic (older format))
At the start: 42 parts

Commit message: naming changes
Parts:
- U?: symbol powersupply_version_1:RFM-0505S -> powersupply:RFM-0505S
- U?: symbol powersupply_version_1:TFT_LCD -> powersupply:TFT_LCD
- U?: symbol powersupply_version_1:MC33063AP1 -> powersupply:MC33063AP1
- U?: symbol powersupply_version_1:1x2Pinheader -> powersupply:1x2Pinheader
- U? (x2): symbol powersupply_version_1:LM358P -> powersupply:LM358P
Changed lines of the file:
@@
 EESchema Schematic File Version 4
-LIBS:powersupply_version_1 2-cache
+LIBS:powersupply-cache
 EELAYER 29 0
 EELAYER END
@@
 NoConn ~ 1950 1550
 $Comp
-L powersupply_version_1:RFM-0505S U?
+L powersupply:RFM-0505S U?
 U 1 1 5D303F43
 P 2800 900
@@
 	2550 1150 2550 1200
 $Comp
-L powersupply_version_1:TFT_LCD U?
+L powersupply:TFT_LCD U?
 U 1 1 5D37FF21
 P 5150 4850
@@
 NoConn ~ 25200 10700
 $Comp
-L powersupply_version_1:MC33063AP1 U?
+L powersupply:MC33063AP1 U?
 U 1 1 5D455E56
 P 5900 1400
@@
 Ref_Amustfigureoutwhattodowiththis
 $Comp
-L powersupply_version_1:LM358P U?
+L powersupply:LM358P U?
 U 1 1 5D4A8FA5
 P 8400 3150
@@
 $EndComp
 $Comp
-L powersupply_version_1:LM358P U?
+L powersupply:LM358P U?
 U 1 1 5D4AA099
 P 8400 4300
@@
 Connection ~ 9700 5550
 $Comp
-L powersupply_version_1:1x2Pinheader U?
+L powersupply:1x2Pinheader U?
 U 1 1 5D48A8A7
 P 10850 3850

Commit message: basic changes
Parts:
- removed C? (x2): C_Small, symbol Device:C_Small
- removed J?: Conn_01x05, symbol Connector_Generic:Conn_01x05
- removed RV? (x2): R_POT, symbol Device:R_POT
- removed Y?: Crystal_Small, symbol Device:Crystal_Small
- added C?: 1uF, symbol Device:C_Small
- added J?: Conn_01x02, symbol Connector_Generic:Conn_01x02
- added L?: 170uH, symbol Device:L_Small
- added R? (x5): 1k, symbol Device:R_Small_US
- added U?: joystick-K1-1506DN-01, symbol powersupply:joystick-K1-1506DN-01
- C?: value CP1_Small -> 100uF
- C?: value CP1_Small -> 330uF
- C?: value CP1_Small -> 1500pF
- C? (x2): value C_Small -> 1uF
- C? (x2): value C_Small -> 15uF
- D?: value D_Zener_Small -> 1N5819
- D?: value D_Small -> 1N5819
- R?: value R_Small_US -> 180
- R?: value R_Small_US -> 0.22
- R?: value 1k -> 3.6k
- R?: value 677 -> 5.5k
- R?: value R_Small_US -> 15k
- R? (x2): value R_Small_US -> 100
- R?: value R_Small_US -> 3k
- R?: value R_Small_US -> 132k
- R? (x3): value R_Small_US -> 1k
- R?: value R_Small_US -> 4.7k
- R?: value R_Small_US -> 0.05
- U?: value AZ1117-3.3 -> AZ1117E-3.3
- U?: value 1x2Pinheader -> 1x2
Connections:
- net labels added: SDA, SWDIO, center, down, left, right, up
- net labels removed: Boost_in, CS, Current_set, DC, MISO, MOSI, Ref, Ref_Amustfigureoutwhattodowiththis, Reset, VCC, Voltage_set, mayhavetogroundthese
- wire segments 90 -> 93
- no-connect marks 10 -> 5
Other:
- moved on the sheet: C?, R?, SW?, U?

Commit message: small change
Parts:
- removed U?: LM358P, symbol powersupply:LM358P
Connections:
- wire segments 93 -> 92
Changed lines of the file:
@@
-$EndComp
-$Comp
-L powersupply:LM358P U?
-U 1 1 5D4AA099
-P 8400 4300
-F 0 "U?" H 8375 4415 50  0000 C CNN
-F 1 "LM358P" H 8375 4324 50  0000 C CNN
-F 2 "" H 8400 4300 50  0001 C CNN
-F 3 "" H 8400 4300 50  0001 C CNN
-	1    8400 4300
-	1    0    0    -1
 $EndComp
 $Comp
@@
 	1    0    0    -1
 $EndComp
-$Comp
-L Device:R_Small_US R?
-U 1 1 5D4C174A
-P 8450 5600
-F 0 "R?" V 8650 5600 50  0000 C CNN
-F 1 "100" V 8550 5600 50  0000 C CNN
-F 2 "" H 8450 5600 50  0001 C CNN
-F 3 "~" H 8450 5600 50  0001 C CNN
-	1    8450 5600
-	0    -1   -1   0
-$EndComp
 Wire Wire Line
 	8050 3600 7950 3600
@@
 Wire Wire Line
 	9050 4650 9050 5100
-Wire Wire Line
-	9050 5100 7900 5100
 Wire Wire Line
 	7900 5100 7900 4750
@@
 Connection ~ 8700 3750
 Connection ~ 8700 3600
-Wire Wire Line
-	8700 4600 8700 4750
-Wire Wire Line
-	8700 4900 8700 4750
-Connection ~ 8700 4750
 $Comp
 L power:GND #PWR?
@@
 	1    0    0    -1
 $EndComp
-Connection ~ 8700 4900
 $Comp
 L Device:L_Small L?
@@
 Wire Wire Line
 	7500 5600 7800 5600
-Connection ~ 7800 5600
-Wire Wire Line
-	7800 5600 8350 5600
-Wire Wire Line
-	8550 5600 9200 5600
-Connection ~ 9200 5600
 Wire Wire Line
 	10200 4900 10200 5600
@@
 Wire Wire Line
 	6600 2050 6800 2050
+Connection ~ 9200 5600
+Wire Wire Line
+	8550 5600 9200 5600
+Connection ~ 7800 5600
+Wire Wire Line
+	7800 5600 8350 5600
+Wire Wire Line
+	9050 5100 7900 5100
+$Comp
+L Device:R_Small_US R?
+U 1 1 5D4C174A
+P 8450 5600
+F 0 "R?" V 8650 5600 50  0000 C CNN
+F 1 "100" V 8550 5600 50  0000 C CNN
+F 2 "" H 8450 5600 50  0001 C CNN
+F 3 "~" H 8450 5600 50  0001 C CNN
+	1    8450 5600
+	0    -1   -1   0
+$EndComp
+Wire Wire Line
+	8700 4600 8700 4900
 $EndSCHEMATC

Commit message: big change
Parts:
- removed C?: 100nF, symbol Device:C_Small
- removed J?: Conn_01x02, symbol Connector_Generic:Conn_01x02
- removed R? (x5): 1k, symbol Device:R_Small_US
- added C4, C5: 100uF, symbol Device:CP1_Small
- added D3: 6V, symbol Device:D_Zener_Small
- added J1: Conn_01x03, symbol Connector_Generic:Conn_01x03
- added L2: 1uH, symbol Device:L_Small
- added R101, R104, R105: 4.7k, Resistor_SMD:R_0805_2012Metric, symbol Device:R_Small_US
- added R106, R107, R108, R109: 0, Resistor_SMD:R_0805_2012Metric, symbol Device:R_Small_US
- added R14: 1k, Resistor_THT:R_Axial_DIN0207_L6.3mm_D2.5mm_P10.16mm_Horizontal, symbol Device:R_Small_US
- added R15: 10k, Resistor_THT:R_Axial_DIN0207_L6.3mm_D2.5mm_P10.16mm_Horizontal, symbol Device:R_Small_US
- added R16: 100, Resistor_THT:R_Axial_DIN0207_L6.3mm_D2.5mm_P10.16mm_Horizontal, symbol Device:R_Small_US
- added U10: MCP6001-OT, Package_TO_SOT_SMD:SOT-23-5, symbol Amplifier_Operational:MCP6001-OT
- added U8: 1x2, symbol Connector_Generic:Conn_01x02
- C1: renamed from C?; value 100uF -> 330 uF
- C101, C102, C103, C104, C105: renamed from C?; footprint (none) -> Capacitor_SMD:C_0805_2012Metric
- R1, R10, R13, R2, R3, R4, R5, R6, R7, R8, R9: renamed from R?; footprint (none) -> Resistor_THT:R_Axial_DIN0207_L6.3mm_D2.5mm_P10.16mm_Horizontal
- R102, R103: renamed from R?; footprint (none) -> Resistor_SMD:R_0805_2012Metric
- R11: renamed from R?; value 1k -> 2.32k; footprint (none) -> Resistor_THT:R_Axial_DIN0207_L6.3mm_D2.5mm_P10.16mm_Horizontal
- R12: renamed from R?; value 4.7k -> 1k; footprint (none) -> Resistor_THT:R_Axial_DIN0207_L6.3mm_D2.5mm_P10.16mm_Horizontal
- SW1: renamed from SW?; footprint (none) -> Button_Switch_THT:SW_PUSH_6mm
- U1: renamed from U?; footprint (none) -> Package_TO_SOT_SMD:SOT-223-3_TabPin2
- U3: renamed from U?; value RFM-0505S -> B0505S-2WR2
- U4: renamed from U?; value TFT_LCD -> TFT_OLED; symbol powersupply:TFT_LCD -> powersupply:TFT_OLED
- U9: renamed from U?; symbol powersupply:1x2Pinheader -> Connector_Generic:Conn_01x02
- gave numbers to parts that had none: 11
Connections:
- net labels added: V_boost_ctrl, V_curr_lim, V_current_amplified, V_lin_ctrl, V_negative_out, V_positive_out
- net labels removed: DAC, negative_output, positive_output
- wire segments 92 -> 99
Other:
- moved on the sheet: C1, C103, C104, C105, C2, C3, D1, D2, L1, R1, R10, R102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

Commit message: lib
Parts:
- U2: symbol MCU_Microchip_SAMD:ATSAMD10D13A-SS -> powersupply:ATSAMD10D13A-SS
Other:
- moved on the sheet: C103, C104, C105, R102, R103, U2
Changed lines of the file:
@@
 Connection ~ 2750 2950
 $Comp
-L MCU_Microchip_SAMD:ATSAMD10D13A-SS U2
+L powersupply:ATSAMD10D13A-SS U2
 U 1 1 5D47B7D4
-P 2500 4650
-F 0 "U2" H 1550 4350 50  0000 C CNN
-F 1 "ATSAMD10D13A-SS" H 1500 4200 50  0000 C CNN
-F 2 "Package_SO:SOIC-20W_7.5x12.8mm_P1.27mm" H 2500 3500 50  0001 C CNN
-F 3 "http://ww1.microchip.com/downloads/en/DeviceDoc/Atmel-42242-SAM-D10_Datasheet.pdf" H 2500 3750 50  0001 C CNN
-	1    2500 4650
+P 2600 4450
+F 0 "U2" H 1650 4150 50  0000 C CNN
+F 1 "ATSAMD10D13A-SS" H 1600 4000 50  0000 C CNN
+F 2 "Package_SO:SOIC-20W_7.5x12.8mm_P1.27mm" H 2600 3300 50  0001 C CNN
+F 3 "http://ww1.microchip.com/downloads/en/DeviceDoc/Atmel-42242-SAM-D10_Datasheet.pdf" H 2600 3550 50  0001 C CNN
+	1    2600 4450
 	1    0    0    -1
 $EndComp
@@
 L Device:R_Small_US R103
 U 1 1 5D4F946F
-P 3350 5150
-F 0 "R103" V 3145 5150 50  0000 C CNN
-F 1 "1k" V 3236 5150 50  0000 C CNN
-F 2 "Resistor_SMD:R_0805_2012Metric" H 3350 5150 50  0001 C CNN
-F 3 "~" H 3350 5150 50  0001 C CNN
-	1    3350 5150
+P 3350 6250
+F 0 "R103" V 3145 6250 50  0000 C CNN
+F 1 "1k" V 3236 6250 50  0000 C CNN
+F 2 "Resistor_SMD:R_0805_2012Metric" H 3350 6250 50  0001 C CNN
+F 3 "~" H 3350 6250 50  0001 C CNN
+	1    3350 6250
 	0    1    1    0
 $EndComp
@@
 L Device:R_Small_US R102
 U 1 1 5D4FAA70
-P 3100 5250
-F 0 "R102" V 3200 5250 50  0000 C CNN
-F 1 "1k" V 3300 5250 50  0000 C CNN
-F 2 "Resistor_SMD:R_0805_2012Metric" H 3100 5250 50  0001 C CNN
-F 3 "~" H 3100 5250 50  0001 C CNN
-	1    3100 5250
+P 3100 6450
+F 0 "R102" V 3200 6450 50  0000 C CNN
+F 1 "1k" V 3300 6450 50  0000 C CNN
+F 2 "Resistor_SMD:R_0805_2012Metric" H 3100 6450 50  0001 C CNN
+F 3 "~" H 3100 6450 50  0001 C CNN
+	1    3100 6450
 	0    1    1    0
 $EndComp
@@
 L Device:C_Small C103
 U 1 1 5D502474
-P 3200 5650
-F 0 "C103" H 3292 5696 50  0000 L CNN
-F 1 "15uF" H 3292 5605 50  0000 L CNN
-F 2 "Capacitor_SMD:C_0805_2012Metric" H 3200 5650 50  0001 C CNN
-F 3 "~" H 3200 5650 50  0001 C CNN
-	1    3200 5650
-	1    0    0    -1
-$EndComp
-Text Label 3200 5350 0    50   ~ 0
+P 3200 6850
+F 0 "C103" H 3292 6896 50  0000 L CNN
+F 1 "15uF" H 3292 6805 50  0000 L CNN
+F 2 "Capacitor_SMD:C_0805_2012Metric" H 3200 6850 50  0001 C CNN
+F 3 "~" H 3200 6850 50  0001 C CNN
+	1    3200 6850
+	1    0    0    -1
+$EndComp
+Text Label 3200 6650 0    50   ~ 0
 V_curr_lim
-Text Label 3650 5250 0    50   ~ 0
+Text Label 3650 6350 0    50   ~ 0
 V_boost_ctrl
-Text Label 3000 4950 0    50   ~ 0
+Text Label 3000 5850 0    50   ~ 0
 SDA
 $Comp
@@
 $EndComp
 Wire Wire Line
-	3200 5250 3200 5550
-Wire Wire Line
-	3000 5150 3250 5150
-Wire Wire Line
-	3450 5150 3650 5150
-Wire Wire Line
-	3650 5150 3650 5300
+	3200 6450 3200 6750
+Wire Wire Line
+	3000 6250 3250 6250
+Wire Wire Line
+	3450 6250 3650 6250
+Wire Wire Line
+	3650 6250 3650 6400
 $Comp
 L Regulator_Linear:AZ1117-3.3 U1
@@
 L Device:C_Small C105
 U 1 1 5D5092B9
-P 3650 5400
-F 0 "C105" H 3742 5446 50  0000 L CNN
-F 1 "15uF" H 3742 5355 50  0000 L CNN
-F 2 "Capacitor_SMD:C_0805_2012Metric" H 3650 5400 50  0001 C CNN
-F 3 "~" H 3650 5400 50  0001 C CNN
-	1    3650 5400
+P 3650 6500
+F 0 "C105" H 3742 6546 50  0000 L CNN
+F 1 "15uF" H 3742 6455 50  0000 L CNN
+F 2 "Capacitor_SMD:C_0805_2012Metric" H 3650 6500 50  0001 C CNN
+F 3 "~" H 3650 6500 50  0001 C CNN
+	1    3650 6500
 	1    0    0    -1
 $EndComp
@@
 L power:GND #PWR0126
 U 1 1 5D67264E
-P 2500 5450
-F 0 "#PWR0126" H 2500 5200 50  0001 C CNN
-F 1 "GND" H 2505 5277 50  0000 C CNN
-F 2 "" H 2500 5450 50  0001 C CNN
-F 3 "" H 2500 5450 50  0001 C CNN
-	1    2500 5450
+P 2450 6600
+F 0 "#PWR0126" H 2450 6350 50  0001 C CNN
+F 1 "GND" H 2455 6427 50  0000 C CNN
+F 2 "" H 2450 6600 50  0001 C CNN
+F 3 "" H 2450 6600 50  0001 C CNN
+	1    2450 6600
 	1    0    0    -1
 $EndComp
@@
 L power:GND #PWR0127
 U 1 1 5D673041
-P 3200 5750
-F 0 "#PWR0127" H 3200 5500 50  0001 C CNN
-F 1 "GND" H 3205 5577 50  0000 C CNN
-F 2 "" H 3200 5750 50  0001 C CNN
-F 3 "" H 3200 5750 50  0001 C CNN
-	1    3200 5750
+P 3200 6950
+F 0 "#PWR0127" H 3200 6700 50  0001 C CNN
+F 1 "GND" H 3205 6777 50  0000 C CNN
+F 2 "" H 3200 6950 50  0001 C CNN
+F 3 "" H 3200 6950 50  0001 C CNN
+	1    3200 6950
 	1    0    0    -1
 $EndComp
@@
 L power:GND #PWR0128
 U 1 1 5D673BAE
-P 3650 5500
-F 0 "#PWR0128" H 3650 5250 50  0001 C CNN
-F 1 "GND" H 3655 5327 50  0000 C CNN
-F 2 "" H 3650 5500 50  0001 C CNN
-F 3 "" H 3650 5500 50  0001 C CNN
-	1    3650 5500
-	1    0    0    -1
-$EndComp
-Text Label 2000 4550 2    50   ~ 0
+P 3650 6600
+F 0 "#PWR0128" H 3650 6350 50  0001 C CNN
+F 1 "GND" H 3655 6427 50  0000 C CNN
+F 2 "" H 3650 6600 50  0001 C CNN
+F 3 "" H 3650 6600 50  0001 C CNN
+	1    3650 6600
+	1    0    0    -1
+$EndComp
+Text Label 2000 4650 2    50   ~ 0
 SWDIO
 Text Label 1250 5650 2    50   ~ 0
@@
 	1    0    0    -1
 $EndComp
-Text Label 3000 4450 0    50   ~ 0
+Text Label 3000 4850 0    50   ~ 0
 up
-Text Label 3000 4550 0    50   ~ 0
+Text Label 3000 5050 0    50   ~ 0
 left
+Text Label 3000 5250 0    50   ~ 0
+down
 Text Label 3000 4650 0    50   ~ 0
-down
-Text Label 3000 4350 0    50   ~ 0
 center
 Text Label 5400 5800 2    50   ~ 0
@@
 L power:+3.3V #PWR0136
 U 1 1 5D5A1ADB
-P 3450 4150
-F 0 "#PWR0136" H 3450 4000 50  0001 C CNN
-F 1 "+3.3V" H 3465 4323 50  0000 C CNN
-F 2 "" H 3450 4150 50  0001 C CNN
-F 3 "" H 3450 4150 50  0001 C CNN
-	1    3450 4150
+P 3450 4250
+F 0 "#PWR0136" H 3450 4100 50  0001 C CNN
+F 1 "+3.3V" H 3465 4423 50  0000 C CNN
+F 2 "" H 3450 4250 50  0001 C CNN
+F 3 "" H 3450 4250 50  0001 C CNN
+	1    3450 4250
 	1    0    0    -1
 $EndComp
@@
 L power:GND #PWR0137
 U 1 1 5D5A24F1
-P 4050 4150
-F 0 "#PWR0137" H 4050 3900 50  0001 C CNN
-F 1 "GND" H 4055 3977 50  0000 C CNN
-F 2 "" H 4050 4150 50  0001 C CNN
-F 3 "" H 4050 4150 50  0001 C CNN
-	1    4050 4150
+P 4050 4250
+F 0 "#PWR0137" H 4050 4000 50  0001 C CNN
+F 1 "GND" H 4055 4077 50  0000 C CNN
+F 2 "" H 4050 4250 50  0001 C CNN
+F 3 "" H 4050 4250 50  0001 C CNN
+	1    4050 4250
 	1    0    0    -1
 $EndComp
@@
 L Device:C_Small C104
 U 1 1 5D5A2D7A
-P 3800 4150
-F 0 "C104" V 3571 4150 50  0000 C CNN
-F 1 "1uF" V 3662 4150 50  0000 C CNN
-F 2 "Capacitor_SMD:C_0805_2012Metric" H 3800 4150 50  0001 C CNN
-F 3 "~" H 3800 4150 50  0001 C CNN
-	1    3800 4150
+P 3800 4250
+F 0 "C104" V 3571 4250 50  0000 C CNN
+F 1 "1uF" V 3662 4250 50  0000 C CNN
+F 2 "Capacitor_SMD:C_0805_2012Metric" H 3800 4250 50  0001 C CNN
+F 3 "~" H 3800 4250 50  0001 C CNN
+	1    3800 4250
 	0    1    1    0
 $EndComp
 Wire Wire Line
-	3450 4150 3700 4150
-Connection ~ 3450 4150
-Wire Wire Line
-	3900 4150 4050 4150
+	3450 4250 3700 4250
+Connection ~ 3450 4250
+Wire Wire Line
+	3900 4250 4050 4250
 $Comp
 L Device:R_Small_US R101
@@
 U 1 1 5D5E94BA
 P 7750 5750
-F 0 "U10" H 7750 5269 50  0000 C CNN
-F 1 "MCP6001-OT" H 7750 5360 50  0000 C CNN
+F 0 "U10" H 7950 6100 50  0000 C CNN
+F 1 "MCP6001-OT" H 7950 6000 50  0000 C CNN
 F 2 "Package_TO_SOT_SMD:SOT-23-5" H 7650 5550 50  0001 L CNN
 F 3 "http://ww1.microchip.com/downloads/en/DeviceDoc/21733j.pdf" H 7750 5950 50  0001 C CNN
@@
 	1    0    0    -1
 $EndComp
-Text Label 3000 4250 0    50   ~ 0
+Text Label 3000 4450 0    50   ~ 0
 V_current_amplified
-Text Label 3000 4850 0    50   ~ 0
+Text Label 3000 5650 0    50   ~ 0
 V_positive_out
 Text Label 6800 4250 0    50   ~ 0
@@
 	6600 4250 6800 4250
 Connection ~ 6600 4250
-Text Label 3000 5050 0    50   ~ 0
+Text Label 3000 6050 0    50   ~ 0
 SCK
 $Comp
@@
 	6600 4650 6800 4650
 Connection ~ 6600 4650
-Text Label 3000 4750 0    50   ~ 0
+Text Label 3000 5450 0    50   ~ 0
 right
 Wire Wire Line
@@
 $EndComp
 Wire Wire Line
-	3000 4150 3450 4150
+	3000 4250 3450 4250
 $EndSCHEMATC

Commit message: nothing...
Parts:
- J1: footprint (none) -> Connector_PinHeader_2.54mm:PinHeader_1x03_P2.54mm_Vertical
Changed lines of the file:
@@
 F 0 "J1" H 1530 5792 50  0000 L CNN
 F 1 "Conn_01x03" H 1530 5701 50  0000 L CNN
-F 2 "" H 1450 5750 50  0001 C CNN
+F 2 "Connector_PinHeader_2.54mm:PinHeader_1x03_P2.54mm_Vertical" H 1450 5750 50  0001 C CNN
 F 3 "~" H 1450 5750 50  0001 C CNN
 	1    1450 5750

Commit message: Footprints added
Parts:
- removed C2: 1500pF, symbol Device:CP1_Small
- removed D1: 1N5819, symbol Device:D_Zener_Small
- removed D2: 1N5819, symbol Device:D_Small
- added C2: 1500pF, Capacitor_THT:C_Rect_L4.0mm_W2.5mm_P2.50mm, symbol Device:C_Small
- added D1, D2: 1N5819, Diode_THT:D_DO-41_SOD81_P7.62mm_Horizontal, symbol Device:D_Schottky_Small
- C1: value 330 uF -> 330uF; footprint (none) -> Capacitor_THT:CP_Radial_D10.0mm_P5.00mm
- C3, C4, C5: footprint (none) -> Capacitor_THT:CP_Radial_D10.0mm_P5.00mm
- D3: footprint (none) -> Diode_THT:D_DO-201AE_P15.24mm_Horizontal
- J2: footprint (none) -> powersupply:USB_Micro-B_Amphenol_10118194-0001LF_Horizontal
- L1, L2: footprint (none) -> Inductor_THT:L_Axial_L11.0mm_D4.5mm_P15.24mm_Horizontal_Fastron_MECC
- Q1, U4: footprint (none) -> powersupply:IRF9540N-PMOS
- U3: footprint (none) -> powersupply:B0505S-2WR2-Isolator
- U5: footprint (none) -> powersupply:K1-1506DN-01_joystick
- U6: footprint (none) -> Package_SO:SOIC-8_3.9x4.9mm_P1.27mm
- U7: footprint (none) -> powersupply:LM358P
- U8: footprint (none) -> powersupply:Banana Sockets
- U9: footprint (none) -> Connector_PinHeader_2.54mm:PinHeader_1x02_P2.54mm_Vertical
Connections:
- net GND: now also C2.2
- net at L1.2, U6.1 (Sw_coll): now also D1.2 (A)
- net at U6.3 (Timing_cap): now also C2.1
- net at C3.1, L2.1, R5.2: now also D1.1 (K)
- net at U7.1 (Out1): now also D2.2 (A)
- net at Q1.1 (G), R10.1: now also D2.1 (K)
Changed lines of the file:
@@
 F 0 "J2" H 1707 1817 50  0000 C CNN
 F 1 "USB_B_Micro" H 1707 1726 50  0000 C CNN
-F 2 "" H 1800 1300 50  0001 C CNN
+F 2 "powersupply:USB_Micro-B_Amphenol_10118194-0001LF_Horizontal" H 1800 1300 50  0001 C CNN
 F 3 "~" H 1800 1300 50  0001 C CNN
 	1    1650 1350
@@
 F 0 "U3" H 2800 825 50  0000 C CNN
 F 1 "B0505S-2WR2" H 2800 734 50  0000 C CNN
-F 2 "" H 2800 900 50  0001 C CNN
+F 2 "powersupply:B0505S-2WR2-Isolator" H 2800 900 50  0001 C CNN
 F 3 "" H 2800 900 50  0001 C CNN
 	1    2800 900
@@
 F 0 "U7" H 8375 3265 50  0000 C CNN
 F 1 "LM358P" H 8375 3174 50  0000 C CNN
-F 2 "" H 8400 3150 50  0001 C CNN
+F 2 "powersupply:LM358P" H 8400 3150 50  0001 C CNN
 F 3 "" H 8400 3150 50  0001 C CNN
 	1    8400 3150
@@
 	1    7400 3650
 	1    0    0    -1
-$EndComp
-$Comp
-L Device:D_Small D2
-U 1 1 5D4B1412
-P 9100 2900
-F 0 "D2" H 9100 2695 50  0000 C CNN
-F 1 "1N5819" H 9000 2800 50  0000 C CNN
-F 2 "" V 9100 2900 50  0001 C CNN
-F 3 "~" V 9100 2900 50  0001 C CNN
-	1    9100 2900
-	-1   0    0    1
 $EndComp
 Text Label 7400 3250 2    50   ~ 0
@@
 F 0 "U4" H 5600 3850 50  0000 L CNN
 F 1 "TFT_OLED" H 5500 3700 50  0000 L CNN
-F 2 "" H 5650 3850 50  0001 C CNN
+F 2 "powersupply:IRF9540N-PMOS" H 5650 3850 50  0001 C CNN
 F 3 "" H 5650 3850 50  0001 C CNN
 	1    5650 3850
@@
 F 0 "Q1" H 9806 3404 50  0000 L CNN
 F 1 "Q_PMOS_GDS" H 9806 3495 50  0000 L CNN
-F 2 "" H 9800 3550 50  0001 C CNN
+F 2 "powersupply:IRF9540N-PMOS" H 9800 3550 50  0001 C CNN
 F 3 "~" H 9600 3450 50  0001 C CNN
 	1    9600 3450
@@
 F 0 "U5" H 5850 5500 50  0000 C CNN
 F 1 "joystick-K1-1506DN-01" H 5900 5400 50  0000 C CNN
-F 2 "" H 5850 5500 50  0001 C CNN
+F 2 "powersupply:K1-1506DN-01_joystick" H 5850 5500 50  0001 C CNN
 F 3 "" H 5850 5500 50  0001 C CNN
 	1    5850 5500
@@
 F 0 "U6" H 6150 1415 50  0000 C CNN
 F 1 "MC33063AP1" H 6150 1324 50  0000 C CNN
-F 2 "" H 6150 1300 50  0001 C CNN
+F 2 "Package_SO:SOIC-8_3.9x4.9mm_P1.27mm" H 6150 1300 50  0001 C CNN
 F 3 "" H 6150 1300 50  0001 C CNN
 	1    6150 1300
@@
 P 5200 2050
 F 0 "C1" H 4950 2100 50  0000 L CNN
-F 1 "330 uF" H 4850 2000 50  0000 L CNN
-F 2 "" H 5200 2050 50  0001 C CNN
+F 1 "330uF" H 4850 2000 50  0000 L CNN
+F 2 "Capacitor_THT:CP_Radial_D10.0mm_P5.00mm" H 5200 2050 50  0001 C CNN
 F 3 "~" H 5200 2050 50  0001 C CNN
 	1    5200 2050
@@
 F 0 "C3" H 7341 2696 50  0000 L CNN
 F 1 "330uF" H 7341 2605 50  0000 L CNN
-F 2 "" H 7250 2650 50  0001 C CNN
+F 2 "Capacitor_THT:CP_Radial_D10.0mm_P5.00mm" H 7250 2650 50  0001 C CNN
 F 3 "~" H 7250 2650 50  0001 C CNN
 	1    7250 2650
@@
 	-1   0    0    -1
 $EndComp
-$Comp
-L Device:D_Zener_Small D1
-U 1 1 5D470D69
-P 7250 1750
-F 0 "D1" V 7296 1682 50  0000 R CNN
-F 1 "1N5819" V 7205 1682 50  0000 R CNN
-F 2 "" V 7250 1750 50  0001 C CNN
-F 3 "~" V 7250 1750 50  0001 C CNN
-	1    7250 1750
-	0    1    -1   0
-$EndComp
 Wire Wire Line
 	7250 1850 7250 2550
@@
 Wire Wire Line
 	6850 2200 6700 2200
-$Comp
-L Device:CP1_Small C2
-U 1 1 5D4755C0
-P 7100 2050
-F 0 "C2" H 7191 2096 50  0000 L CNN
-F 1 "1500pF" H 7191 2005 50  0000 L CNN
-F 2 "" H 7100 2050 50  0001 C CNN
-F 3 "~" H 7100 2050 50  0001 C CNN
-	1    7100 2050
-	-1   0    0    -1
-$EndComp
 Wire Wire Line
 	7100 1950 6700 1950
@@
 F 0 "L1" V 5719 950 50  0000 C CNN
 F 1 "170uH" V 5810 950 50  0000 C CNN
-F 2 "" H 5900 950 50  0001 C CNN
+F 2 "Inductor_THT:L_Axial_L11.0mm_D4.5mm_P15.24mm_Horizontal_Fastron_MECC" H 5900 950 50  0001 C CNN
 F 3 "~" H 5900 950 50  0001 C CNN
 	1    5900 950
@@
 F 0 "L2" V 7885 2550 50  0000 C CNN
 F 1 "1uH" V 7794 2550 50  0000 C CNN
-F 2 "" H 7700 2550 50  0001 C CNN
+F 2 "Inductor_THT:L_Axial_L11.0mm_D4.5mm_P15.24mm_Horizontal_Fastron_MECC" H 7700 2550 50  0001 C CNN
 F 3 "~" H 7700 2550 50  0001 C CNN
 	1    7700 2550
@@
 F 0 "C4" H 7891 2696 50  0000 L CNN
 F 1 "100uF" H 7891 2605 50  0000 L CNN
-F 2 "" H 7800 2650 50  0001 C CNN
+F 2 "Capacitor_THT:CP_Radial_D10.0mm_P5.00mm" H 7800 2650 50  0001 C CNN
 F 3 "~" H 7800 2650 50  0001 C CNN
 	1    7800 2650
@@
 F 0 "U9" H 10200 3850 50  0000 L CNN
 F 1 "1x2" H 10200 3950 50  0000 L CNN
-F 2 "" H 10300 4600 50  0001 C CNN
+F 2 "Connector_PinHeader_2.54mm:PinHeader_1x02_P2.54mm_Vertical" H 10300 4600 50  0001 C CNN
 F 3 "" H 10300 4600 50  0001 C CNN
 	1    10300 4450
@@
 F 0 "C5" H 9991 4296 50  0000 L CNN
 F 1 "100uF" H 9991 4205 50  0000 L CNN
-F 2 "" H 9900 4250 50  0001 C CNN
+F 2 "Capacitor_THT:CP_Radial_D10.0mm_P5.00mm" H 9900 4250 50  0001 C CNN
 F 3 "~" H 9900 4250 50  0001 C CNN
 	1    9900 4250
@@
 	0    1    1    0
 $EndComp
-$Comp
-L Device:D_Zener_Small D3
-U 1 1 5D5DCC75
-P 3450 1250
-F 0 "D3" H 3450 1455 50  0000 C CNN
-F 1 "6V" H 3450 1364 50  0000 C CNN
-F 2 "" V 3450 1250 50  0001 C CNN
-F 3 "~" V 3450 1250 50  0001 C CNN
-	1    3450 1250
-	1    0    0    -1
-$EndComp
 Wire Wire Line
 	3350 1250 3050 1250
@@
 F 0 "U8" H 10550 3850 50  0000 L CNN
 F 1 "1x2" H 10550 3950 50  0000 L CNN
-F 2 "" H 10650 4600 50  0001 C CNN
+F 2 "powersupply:Banana Sockets" H 10650 4600 50  0001 C CNN
 F 3 "" H 10650 4600 50  0001 C CNN
 	1    10650 4450
@@
 Wire Wire Line
 	3000 4250 3450 4250
+$Comp
+L Device:C_Small C2
+U 1 1 5D4C7F8E
+P 7100 2050
+F 0 "C2" H 6950 2100 50  0000 L CNN
+F 1 "1500pF" H 6700 2000 50  0000 L CNN
+F 2 "Capacitor_THT:C_Rect_L4.0mm_W2.5mm_P2.50mm" H 7100 2050 50  0001 C CNN
+F 3 "~" H 7100 2050 50  0001 C CNN
+	1    7100 2050
+	1    0    0    -1
+$EndComp
+$Comp
+L Device:D_Schottky_Small D2
+U 1 1 5D4E566E
+P 9100 2900
+F 0 "D2" H 9100 2695 50  0000 C CNN
+F 1 "1N5819" H 9100 2786 50  0000 C CNN
+F 2 "Diode_THT:D_DO-41_SOD81_P7.62mm_Horizontal" V 9100 2900 50  0001 C CNN
+F 3 "~" V 9100 2900 50  0001 C CNN
+	1    9100 2900
+	-1   0    0    1
+$EndComp
+$Comp
+L Device:D_Schottky_Small D1
+U 1 1 5D4EED9B
+P 7250 1750
+F 0 "D1" V 7296 1682 50  0000 R CNN
+F 1 "1N5819" V 7205 1682 50  0000 R CNN
+F 2 "Diode_THT:D_DO-41_SOD81_P7.62mm_Horizontal" V 7250 1750 50  0001 C CNN
+F 3 "~" V 7250 1750 50  0001 C CNN
+	1    7250 1750
+	0    -1   -1   0
+$EndComp
+$Comp
+L Device:D_Zener_Small D3
+U 1 1 5D4FADCE
+P 3450 1250
+F 0 "D3" H 3450 1455 50  0000 C CNN
+F 1 "6V" H 3450 1364 50  0000 C CNN
+F 2 "Diode_THT:D_DO-201AE_P15.24mm_Horizontal" V 3450 1250 50  0001 C CNN
+F 3 "~" V 3450 1250 50  0001 C CNN
+	1    3450 1250
+	1    0    0    -1
+$EndComp
 $EndSCHEMATC
