File: Power_Supply/powersupply/powersupply.sch (KiCad schematic (older format))
At the start: 54 parts, among them J1 Conn_01x03, J2 USB_B_Micro, Q1 Q_PMOS_GDS, SW1 SW_Push, U1 AZ1117E-3.3, U10 MCP6001-OT, U2 ATSAMD10D13A-SS, U3 B0505S-2WR2, U4 TFT_OLED, U5 joystick-K1-1506DN-01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

Commit message: layout changes
Parts:
- U4: footprint powersupply:IRF9540N-PMOS -> powersupply:TFT_OLED_display
Changed lines of the file:
@@
 F 0 "U4" H 5600 3850 50  0000 L CNN
 F 1 "TFT_OLED" H 5500 3700 50  0000 L CNN
-F 2 "powersupply:IRF9540N-PMOS" H 5650 3850 50  0001 C CNN
+F 2 "powersupply:TFT_OLED_display" H 5650 3850 50  0001 C CNN
 F 3 "" H 5650 3850 50  0001 C CNN
 	1    5650 3850
