File: Power_Supply/powersupply/powersupply.sch (KiCad schematic (older format))
At the start: 54 parts, among them J1 Conn_01x03, J2 USB_B_Micro, Q1 Q_PMOS_GDS, SW1 SW_Push, U1 AZ1117E-3.3, U10 MCP6001-OT, U2 ATSAMD10D13A-SS, U3 B0505S-2WR2, U4 TFT_OLED, U5 joystick-K1-1506DN-01, U6 MC33063AP1, U7 LM358P, U8 1x2, U9 1x2

Commit message: more layout
Connections:
- net Vlim is gone; now on net V_lin_ctrl: R6.1
- net Boost_out: no longer C5.1, Q1.2 (D), R11.1, U2.8 (PA16), U8.2 (Pin_2), U9.2 (Pin_2)
- new net V_positive_out: C5.1, Q1.2 (D), R11.1, U2.8 (PA16), U8.2 (Pin_2), U9.2 (Pin_2)
Changed lines of the file:
@@
 $EndComp
 Text Label 7400 3250 2    50   ~ 0
-Vlim
+V_lin_ctrl
 Wire Wire Line
 	8050 2900 8050 3300
@@
 	9050 3750 9050 4100
 Wire Wire Line
-	9700 3250 9700 3650
-Wire Wire Line
 	9700 3650 9700 3750
-Connection ~ 9700 3650
 $Comp
 L power:+5V #PWR0113

Commit message: even more layout
Parts:
- added H1, H2, H3, H4: MountingHole, MountingHole:MountingHole_3.2mm_M3, symbol Mechanical:MountingHole
- added TP1: Boost_out, Connector_PinSocket_2.54mm:PinSocket_1x01_P2.54mm_Vertical, symbol Connector:TestPoint
- added TP2: +5_isolated, Connector_PinSocket_2.54mm:PinSocket_1x01_P2.54mm_Vertical, symbol Connector:TestPoint
- added TP3: +3.3, Connector_PinSocket_2.54mm:PinSocket_1x01_P2.54mm_Vertical, symbol Connector:TestPoint
- added TP4: Current_limit, Connector_PinSocket_2.54mm:PinSocket_1x01_P2.54mm_Vertical, symbol Connector:TestPoint
- added TP5: Voltage_limit, Connector_PinSocket_2.54mm:PinSocket_1x01_P2.54mm_Vertical, symbol Connector:TestPoint
- added TP6: Boost_ctrl, Connector_PinSocket_2.54mm:PinSocket_1x01_P2.54mm_Vertical, symbol Connector:TestPoint
- added TP7: GND, Connector_PinSocket_2.54mm:PinSocket_1x01_P2.54mm_Vertical, symbol Connector:TestPoint
Connections:
- net Vref is gone; now on net V_boost_ctrl: R1.1
- net +3V3: now also TP3.1
- net +5V: now also TP2.1
- net Boost_out: now also TP1.1
- net GND: now also TP7.1
- net V_boost_ctrl: now also TP6.1
- net V_curr_lim: now also R6.1
- net V_lin_ctrl: no longer R6.1
- net Current_limit_divider: now reaches R6.2, R7.1, U7.2 (In1-)
- net Current_limit_divider: now also TP4.1
- net Voltage_limit_divider: now reaches R11.2, R12.1, U7.8 (In2+)
- net Voltage_limit_divider: now also TP5.1
Changed lines of the file:
@@
 $EndComp
 Text Label 7400 3250 2    50   ~ 0
-V_lin_ctrl
+V_curr_lim
 Wire Wire Line
 	8050 2900 8050 3300
@@
 	5500 2550 5100 2550
 Text Label 4900 2550 2    50   ~ 0
-Vref
+V_boost_ctrl
 $Comp
 L power:+5V #PWR0138
@@
 	1    0    0    -1
 $EndComp
+$Comp
+L Connector:TestPoint TP3
+U 1 1 5D4B6929
+P 9450 950
+F 0 "TP3" H 9392 976 50  0000 R CNN
+F 1 "+3.3" H 9392 1067 50  0000 R CNN
+F 2 "Connector_PinSocket_2.54mm:PinSocket_1x01_P2.54mm_Vertical" H 9650 950 50  0001 C CNN
+F 3 "~" H 9650 950 50  0001 C CNN
+	1    9450 950
+	-1   0    0    1
+$EndComp
+$Comp
+L Connector:TestPoint TP2
+U 1 1 5D4B73A5
+P 9900 950
+F 0 "TP2" H 9842 976 50  0000 R CNN
+F 1 "+5_isolated" H 9842 1067 50  0000 R CNN
+F 2 "Connector_PinSocket_2.54mm:PinSocket_1x01_P2.54mm_Vertical" H 10100 950 50  0001 C CNN
+F 3 "~" H 10100 950 50  0001 C CNN
+	1    9900 950
+	-1   0    0    1
+$EndComp
+$Comp
+L Connector:TestPoint TP1
+U 1 1 5D4B7B24
+P 8700 1750
+F 0 "TP1" H 8758 1868 50  0000 L CNN
+F 1 "Boost_out" H 8758 1777 50  0000 L CNN
+F 2 "Connector_PinSocket_2.54mm:PinSocket_1x01_P2.54mm_Vertical" H 8900 1750 50  0001 C CNN
+F 3 "~" H 8900 1750 50  0001 C CNN
+	1    8700 1750
+	1    0    0    -1
+$EndComp
+$Comp
+L Connector:TestPoint TP4
+U 1 1 5D4B85BC
+P 9600 2250
+F 0 "TP4" H 9658 2368 50  0000 L CNN
+F 1 "Current_limit" H 9658 2277 50  0000 L CNN
+F 2 "Connector_PinSocket_2.54mm:PinSocket_1x01_P2.54mm_Vertical" H 9800 2250 50  0001 C CNN
+F 3 "~" H 9800 2250 50  0001 C CNN
+	1    9600 2250
+	1    0    0    -1
+$EndComp
+Text Label 9400 4100 0    50   ~ 0
+Voltage_limit_divider
+Text Label 9600 2250 2    50   ~ 0
+Current_limit_divider
+$Comp
+L Connector:TestPoint TP5
+U 1 1 5D4BBCE8
+P 8650 2150
+F 0 "TP5" H 8708 2268 50  0000 L CNN
+F 1 "Voltage_limit" H 8708 2177 50  0000 L CNN
+F 2 "Connector_PinSocket_2.54mm:PinSocket_1x01_P2.54mm_Vertical" H 8850 2150 50  0001 C CNN
+F 3 "~" H 8850 2150 50  0001 C CNN
+	1    8650 2150
+	1    0    0    -1
+$EndComp
+Text Label 7400 3450 2    50   ~ 0
+Current_limit_divider
+Text Label 8650 2150 2    50   ~ 0
+Voltage_limit_divider
+$Comp
+L Connector:TestPoint TP6
+U 1 1 5D4BF42E
+P 9950 1500
+F 0 "TP6" H 10008 1618 50  0000 L CNN
+F 1 "Boost_ctrl" H 10008 1527 50  0000 L CNN
+F 2 "Connector_PinSocket_2.54mm:PinSocket_1x01_P2.54mm_Vertical" H 10150 1500 50  0001 C CNN
+F 3 "~" H 10150 1500 50  0001 C CNN
+	1    9950 1500
+	1    0    0    -1
+$EndComp
+Text Label 9950 1500 2    50   ~ 0
+V_boost_ctrl
+Text Label 8700 1750 2    50   ~ 0
+Boost_out
+$Comp
+L Connector:TestPoint TP7
+U 1 1 5D4C0DDA
+P 8850 1250
+F 0 "TP7" H 8908 1368 50  0000 L CNN
+F 1 "GND" H 8908 1277 50  0000 L CNN
+F 2 "Connector_PinSocket_2.54mm:PinSocket_1x01_P2.54mm_Vertical" H 9050 1250 50  0001 C CNN
+F 3 "~" H 9050 1250 50  0001 C CNN
+	1    8850 1250
+	1    0    0    -1
+$EndComp
+$Comp
+L power:GND #PWR0121
+U 1 1 5D4C160D
+P 8850 1250
+F 0 "#PWR0121" H 8850 1000 50  0001 C CNN
+F 1 "GND" H 8855 1077 50  0000 C CNN
+F 2 "" H 8850 1250 50  0001 C CNN
+F 3 "" H 8850 1250 50  0001 C CNN
+	1    8850 1250
+	1    0    0    -1
+$EndComp
+$Comp
+L power:+3.3V #PWR0129
+U 1 1 5D4CD74E
+P 9450 950
+F 0 "#PWR0129" H 9450 800 50  0001 C CNN
+F 1 "+3.3V" H 9465 1123 50  0000 C CNN
+F 2 "" H 9450 950 50  0001 C CNN
+F 3 "" H 9450 950 50  0001 C CNN
+	1    9450 950
+	1    0    0    -1
+$EndComp
+$Comp
+L power:+5V #PWR0130
+U 1 1 5D4CDF6D
+P 9900 950
+F 0 "#PWR0130" H 9900 800 50  0001 C CNN
+F 1 "+5V" H 9915 1123 50  0000 C CNN
+F 2 "" H 9900 950 50  0001 C CNN
+F 3 "" H 9900 950 50  0001 C CNN
+	1    9900 950
+	1    0    0    -1
+$EndComp
+$Comp
+L Mechanical:MountingHole H1
+U 1 1 5D4CE857
+P 3550 2850
+F 0 "H1" H 3650 2896 50  0000 L CNN
+F 1 "MountingHole" H 3650 2805 50  0000 L CNN
+F 2 "MountingHole:MountingHole_3.2mm_M3" H 3550 2850 50  0001 C CNN
+F 3 "~" H 3550 2850 50  0001 C CNN
+	1    3550 2850
+	1    0    0    -1
+$EndComp
+$Comp
+L Mechanical:MountingHole H2
+U 1 1 5D4CF35E
+P 4050 3100
+F 0 "H2" H 4150 3146 50  0000 L CNN
+F 1 "MountingHole" H 4150 3055 50  0000 L CNN
+F 2 "MountingHole:MountingHole_3.2mm_M3" H 4050 3100 50  0001 C CNN
+F 3 "~" H 4050 3100 50  0001 C CNN
+	1    4050 3100
+	1    0    0    -1
+$EndComp
+$Comp
+L Mechanical:MountingHole H3
+U 1 1 5D4CFB63
+P 4650 3300
+F 0 "H3" H 4750 3346 50  0000 L CNN
+F 1 "MountingHole" H 4750 3255 50  0000 L CNN
+F 2 "MountingHole:MountingHole_3.2mm_M3" H 4650 3300 50  0001 C CNN
+F 3 "~" H 4650 3300 50  0001 C CNN
+	1    4650 3300
+	1    0    0    -1
+$EndComp
+$Comp
+L Mechanical:MountingHole H4
+U 1 1 5D4D0374
+P 5900 3300
+F 0 "H4" H 6000 3346 50  0000 L CNN
+F 1 "MountingHole" H 6000 3255 50  0000 L CNN
+F 2 "MountingHole:MountingHole_3.2mm_M3" H 5900 3300 50  0001 C CNN
+F 3 "~" H 5900 3300 50  0001 C CNN
+	1    5900 3300
+	1    0    0    -1
+$EndComp

Commit message: almost finished layout
Connections:
- net V_negative_out: now also U8.2 (Pin_2), U9.2 (Pin_2); no longer U8.1 (Pin_1), U9.1 (Pin_1)
- net V_positive_out: now also U8.1 (Pin_1), U9.1 (Pin_1); no longer U8.2 (Pin_2), U9.2 (Pin_2)
Changed lines of the file:
@@
 L Connector_Generic:Conn_01x02 U9
 U 1 1 5D48A8A7
-P 10300 4450
-F 0 "U9" H 10200 3850 50  0000 L CNN
-F 1 "1x2" H 10200 3950 50  0000 L CNN
-F 2 "Connector_PinHeader_2.54mm:PinHeader_1x02_P2.54mm_Vertical" H 10300 4600 50  0001 C CNN
-F 3 "" H 10300 4600 50  0001 C CNN
-	1    10300 4450
-	-1   0    0    1
+P 10300 4350
+F 0 "U9" H 10200 3750 50  0000 L CNN
+F 1 "1x2" H 10200 3850 50  0000 L CNN
+F 2 "Connector_PinHeader_2.54mm:PinHeader_1x02_P2.54mm_Vertical" H 10300 4500 50  0001 C CNN
+F 3 "" H 10300 4500 50  0001 C CNN
+	1    10300 4350
+	-1   0    0    -1
 $EndComp
 Connection ~ 9900 3750
@@
 	10850 3750 10850 4350
 Connection ~ 10500 3750
-Wire Wire Line
-	10850 4450 10850 5050
 Wire Wire Line
 	10850 5050 10500 5050
@@
 L Connector_Generic:Conn_01x02 U8
 U 1 1 5D4A34EF
-P 10650 4450
-F 0 "U8" H 10550 3850 50  0000 L CNN
-F 1 "1x2" H 10550 3950 50  0000 L CNN
-F 2 "powersupply:Banana Sockets" H 10650 4600 50  0001 C CNN
-F 3 "" H 10650 4600 50  0001 C CNN
-	1    10650 4450
-	-1   0    0    1
+P 10650 4350
+F 0 "U8" H 10550 3750 50  0000 L CNN
+F 1 "1x2" H 10550 3850 50  0000 L CNN
+F 2 "powersupply:Banana Sockets" H 10650 4500 50  0001 C CNN
+F 3 "" H 10650 4500 50  0001 C CNN
+	1    10650 4350
+	-1   0    0    -1
 $EndComp
 Wire Wire Line
@@
 	1    0    0    -1
 $EndComp
+Wire Wire Line
+	10850 4450 10850 5050
 $EndSCHEMATC

Commit message: finalish changes
Parts:
- removed R106, R107, R108, R109: 0, Resistor_SMD:R_0805_2012Metric, symbol Device:R_Small_US
- added R17: 10k, Resistor_THT:R_Axial_DIN0207_L6.3mm_D2.5mm_P10.16mm_Horizontal, symbol Device:R_Small_US
- added TP10, TP11, TP8, TP9: TestPoint, TestPoint:TestPoint_Pad_1.5x1.5mm, symbol Connector:TestPoint
- C1: value 330uF -> 470uF; footprint Capacitor_THT:CP_Radial_D10.0mm_P5.00mm -> Capacitor_THT:CP_Radial_D8.0mm_P3.50mm
- C2: value 1500pF -> 270pF
- C3: value 330uF -> 470u
- C4: value 100uF -> 470u
- L1: value 170uH -> 47uH; footprint Inductor_THT:L_Axial_L11.0mm_D4.5mm_P15.24mm_Horizontal_Fastron_MECC -> Inductor_THT:L_Radial_D8.7mm_P5.00mm_Fastron_07HCP
- R3: value 0.22 -> 0.3 1/4W
- R8: value 132k -> 10k
Connections:
- net +3V3: now also U4.2 (VCC), R17.1, TP10.1, TP8.1
- net +5V: now also D3.1 (K), R14.2, U3.4 (+Vout); no longer D3.2 (A), R14.1
- net Current_limit_divider: now also R17.2
- net GND: now also D3.2 (A), R14.1, U4.1 (GND), TP11.1, TP9.1
- net SCK: now also R105.2, U4.3 (SCK)
- net V_negative_out: no longer U10.3 (+)
- net at R8.2, R9.1, U7.3 (In1+): now also U10.3 (+)
Other:
- moved on the sheet: H1, H2, H3, H4, U5

Commit message: new layout
Parts:
- R11: renamed from R13; value 0.05 -> 0.1
- renumbered R14 to R1, R9 to R10, R17 to R12, R6 to R13, R7 to R14, R10 to R15, R12 to R16, R11 to R17, R3 to R2, R2 to R3, R16 to R4, R15 to R5, R1 to R6, R4 to R7, R5 to R8, R8 to R9
Changed lines of the file:
@@
 $EndComp
 $Comp
-L Device:R_Small_US R6
+L Device:R_Small_US R13
 U 1 1 5D4AC3D3
 P 7400 3350
-F 0 "R6" H 7468 3396 50  0000 L CNN
+F 0 "R13" H 7468 3396 50  0000 L CNN
 F 1 "15k" H 7468 3305 50  0000 L CNN
 F 2 "Resistor_THT:R_Axial_DIN0207_L6.3mm_D2.5mm_P10.16mm_Horizontal" H 7400 3350 50  0001 C CNN
@@
 $EndComp
 $Comp
-L Device:R_Small_US R7
+L Device:R_Small_US R14
 U 1 1 5D4AD799
 P 7400 3550
-F 0 "R7" H 7200 3600 50  0000 L CNN
+F 0 "R14" H 7200 3600 50  0000 L CNN
 F 1 "100" H 7200 3500 50  0000 L CNN
 F 2 "Resistor_THT:R_Axial_DIN0207_L6.3mm_D2.5mm_P10.16mm_Horizontal" H 7400 3550 50  0001 C CNN
@@
 $EndComp
 $Comp
-L Device:R_Small_US R10
+L Device:R_Small_US R15
 U 1 1 5D4B4E12
 P 8950 3450
-F 0 "R10" V 8850 3300 50  0000 L CNN
+F 0 "R15" V 8850 3300 50  0000 L CNN
 F 1 "3k" V 8850 3550 50  0000 L CNN
 F 2 "Resistor_THT:R_Axial_DIN0207_L6.3mm_D2.5mm_P10.16mm_Horizontal" H 8950 3450 50  0001 C CNN
@@
 $EndComp
 $Comp
-L Device:R_Small_US R2
+L Device:R_Small_US R3
 U 1 1 5D459423
 P 5300 1450
-F 0 "R2" V 5095 1450 50  0000 C CNN
+F 0 "R3" V 5095 1450 50  0000 C CNN
 F 1 "180" V 5186 1450 50  0000 C CNN
 F 2 "Resistor_THT:R_Axial_DIN0207_L6.3mm_D2.5mm_P10.16mm_Horizontal" H 5300 1450 50  0001 C CNN
@@
 	5200 1700 5650 1700
 $Comp
-L Device:R_Small_US R3
+L Device:R_Small_US R2
 U 1 1 5D45B2AA
 P 5200 1800
-F 0 "R3" H 5268 1846 50  0000 L CNN
+F 0 "R2" H 5268 1846 50  0000 L CNN
 F 1 "0.3 1/4W" H 5268 1755 50  0000 L CNN
 F 2 "Resistor_THT:R_Axial_DIN0207_L6.3mm_D2.5mm_P10.16mm_Horizontal" H 5200 1800 50  0001 C CNN
@@
 $EndComp
 $Comp
-L Device:R_Small_US R5
+L Device:R_Small_US R8
 U 1 1 5D46B727
 P 5900 2550
-F 0 "R5" V 5695 2550 50  0000 C CNN
+F 0 "R8" V 5695 2550 50  0000 C CNN
 F 1 "5.5k" V 5786 2550 50  0000 C CNN
 F 2 "Resistor_THT:R_Axial_DIN0207_L6.3mm_D2.5mm_P10.16mm_Horizontal" H 5900 2550 50  0001 C CNN
@@
 Boost_out
 $Comp
-L Device:R_Small_US R1
+L Device:R_Small_US R6
 U 1 1 5D49225A
 P 5000 2550
-F 0 "R1" V 4795 2550 50  0000 C CNN
+F 0 "R6" V 4795 2550 50  0000 C CNN
 F 1 "3.17k" V 4886 2550 50  0000 C CNN
 F 2 "Resistor_THT:R_Axial_DIN0207_L6.3mm_D2.5mm_P10.16mm_Horizontal" H 5000 2550 50  0001 C CNN
@@
 Connection ~ 5500 2550
 $Comp
-L Device:R_Small_US R4
+L Device:R_Small_US R7
 U 1 1 5D46A6EF
 P 5500 2650
-F 0 "R4" H 5568 2696 50  0000 L CNN
+F 0 "R7" H 5568 2696 50  0000 L CNN
 F 1 "3.6k" H 5568 2605 50  0000 L CNN
 F 2 "Resistor_THT:R_Axial_DIN0207_L6.3mm_D2.5mm_P10.16mm_Horizontal" H 5500 2650 50  0001 C CNN
@@
 	7250 2550 7600 2550
 $Comp
-L Device:R_Small_US R8
+L Device:R_Small_US R9
 U 1 1 5D4C0D0A
 P 7800 4950
-F 0 "R8" H 7868 4996 50  0000 L CNN
+F 0 "R9" H 7868 4996 50  0000 L CNN
 F 1 "10k" H 7868 4905 50  0000 L CNN
 F 2 "Resistor_THT:R_Axial_DIN0207_L6.3mm_D2.5mm_P10.16mm_Horizontal" H 7800 4950 50  0001 C CNN
@@
 $EndComp
 $Comp
-L Device:R_Small_US R9
+L Device:R_Small_US R10
 U 1 1 5D4C174A
 P 8450 5050
-F 0 "R9" V 8650 5050 50  0000 C CNN
+F 0 "R10" V 8650 5050 50  0000 C CNN
 F 1 "100" V 8550 5050 50  0000 C CNN
 F 2 "Resistor_THT:R_Axial_DIN0207_L6.3mm_D2.5mm_P10.16mm_Horizontal" H 8450 5050 50  0001 C CNN
@@
 $EndComp
 $Comp
-L Device:R_Small_US R11
+L Device:R_Small_US R17
 U 1 1 5D4D044A
 P 9400 3850
-F 0 "R11" H 9468 3896 50  0000 L CNN
+F 0 "R17" H 9468 3896 50  0000 L CNN
 F 1 "2.32k" H 9468 3805 50  0000 L CNN
 F 2 "Resistor_THT:R_Axial_DIN0207_L6.3mm_D2.5mm_P10.16mm_Horizontal" H 9400 3850 50  0001 C CNN
@@
 $EndComp
 $Comp
-L Device:R_Small_US R12
+L Device:R_Small_US R16
 U 1 1 5D4D11A0
 P 9400 4250
-F 0 "R12" H 9468 4296 50  0000 L CNN
+F 0 "R16" H 9468 4296 50  0000 L CNN
 F 1 "1k" H 9468 4205 50  0000 L CNN
 F 2 "Resistor_THT:R_Axial_DIN0207_L6.3mm_D2.5mm_P10.16mm_Horizontal" H 9400 4250 50  0001 C CNN
@@
 	9400 4100 9400 4150
 $Comp
-L Device:R_Small_US R13
+L Device:R_Small_US R11
 U 1 1 5D4E54B6
 P 9200 5150
-F 0 "R13" H 9268 5196 50  0000 L CNN
-F 1 "0.05" H 9268 5105 50  0000 L CNN
+F 0 "R11" H 9268 5196 50  0000 L CNN
+F 1 "0.1" H 9268 5105 50  0000 L CNN
 F 2 "Resistor_THT:R_Axial_DIN0207_L6.3mm_D2.5mm_P10.16mm_Horizontal" H 9200 5150 50  0001 C CNN
 F 3 "~" H 9200 5150 50  0001 C CNN
@@
 Connection ~ 10500 5050
 $Comp
-L Device:R_Small_US R14
+L Device:R_Small_US R1
 U 1 1 5D5DBC0A
 P 3450 1500
-F 0 "R14" V 3250 1500 50  0000 C CNN
+F 0 "R1" V 3250 1500 50  0000 C CNN
 F 1 "1k" V 3336 1500 50  0000 C CNN
 F 2 "Resistor_THT:R_Axial_DIN0207_L6.3mm_D2.5mm_P10.16mm_Horizontal" H 3450 1500 50  0001 C CNN
@@
 	8550 5050 9200 5050
 $Comp
-L Device:R_Small_US R15
+L Device:R_Small_US R5
 U 1 1 5D5F6DCC
 P 7100 5850
-F 0 "R15" H 7168 5896 50  0000 L CNN
+F 0 "R5" H 7168 5896 50  0000 L CNN
 F 1 "10k" H 7168 5805 50  0000 L CNN
 F 2 "Resistor_THT:R_Axial_DIN0207_L6.3mm_D2.5mm_P10.16mm_Horizontal" H 7100 5850 50  0001 C CNN
@@
 $EndComp
 $Comp
-L Device:R_Small_US R16
+L Device:R_Small_US R4
 U 1 1 5D5F7B68
 P 7100 6300
-F 0 "R16" H 7168 6346 50  0000 L CNN
+F 0 "R4" H 7168 6346 50  0000 L CNN
 F 1 "100" H 7168 6255 50  0000 L CNN
 F 2 "Resistor_THT:R_Axial_DIN0207_L6.3mm_D2.5mm_P10.16mm_Horizontal" H 7100 6300 50  0001 C CNN
@@
 $EndComp
 $Comp
-L Device:R_Small_US R17
+L Device:R_Small_US R12
 U 1 1 5D528638
 P 6400 3350
-F 0 "R17" H 6468 3396 50  0000 L CNN
+F 0 "R12" H 6468 3396 50  0000 L CNN
 F 1 "10k" H 6468 3305 50  0000 L CNN
 F 2 "Resistor_THT:R_Axial_DIN0207_L6.3mm_D2.5mm_P10.16mm_Horizontal" H 6400 3350 50  0001 C CNN

Commit message: finalish changes
Parts:
- removed R12, R5: 10k, Resistor_THT:R_Axial_DIN0207_L6.3mm_D2.5mm_P10.16mm_Horizontal, symbol Device:R_Small_US
- removed R4: 100, Resistor_THT:R_Axial_DIN0207_L6.3mm_D2.5mm_P10.16mm_Horizontal, symbol Device:R_Small_US
- removed U10: MCP6001-OT, Package_TO_SOT_SMD:SOT-23-5, symbol Amplifier_Operational:MCP6001-OT
- added C6: C_Small, symbol Device:C_Small
- added D4: C503B 2.1V, symbol Device:LED
- added R18: 300, symbol Device:R_Small_US
- added R19: 18.2k, symbol Device:R_Small_US
- added R20: 4.99k, symbol Device:R_Small_US
- added U10: INA199, symbol powersupply:INA199
- C4: value 470u -> 100u
- D3: footprint Diode_THT:D_DO-201AE_P15.24mm_Horizontal -> Diode_THT:D_DO-35_SOD27_P7.62mm_Horizontal
- R1: value 1k -> 150
- R9: value 10k -> 130k
- SW1: value SW_Push -> KMR2; footprint Button_Switch_THT:SW_PUSH_6mm -> Button_Switch_SMD:SW_Push_1P1T_NO_CK_KMR2
- TP10, TP11, TP8, TP9: footprint TestPoint:TestPoint_Pad_1.5x1.5mm -> powersupply:pads
Connections:
- net +3V3: now also C6.1, U10.3 (V+)
- net +5V: now also R18.1
- net GND: now also SW1.1, C6.2, D4.1 (K), R20.2, U10.1 (Ref), U10.2 (GND), U10.5 (IN-); no longer SW1.2
- net V_boost_ctrl: now also U2.18 (PA02); no longer C105.1, R103.1
- net V_current_amplified: now also U10.6 (OUT)
- net V_lin_ctrl: now also C105.1, R103.1; no longer U2.18 (PA02)
- net V_negative_out: now also U10.4 (IN+)
- net V_positive_out: now also R19.1; no longer U2.8 (PA16)
- net at R101.2, U2.11 (PA28/~RST): now also SW1.2; no longer SW1.1
- new net: R19.2, R20.1, U2.8 (PA16)
- new net: D4.2 (A), R18.2

Commit message: big CHANGES
Parts:
- C3: value 470u -> 470uF; footprint Capacitor_THT:CP_Radial_D10.0mm_P5.00mm -> Capacitor_THT:CP_Radial_D8.0mm_P3.50mm
- C4: value 100u -> 100uF; footprint Capacitor_THT:CP_Radial_D10.0mm_P5.00mm -> Capacitor_THT:CP_Radial_D6.3mm_P2.50mm
- C5: footprint Capacitor_THT:CP_Radial_D10.0mm_P5.00mm -> Capacitor_THT:CP_Radial_D6.3mm_P2.50mm
- C6: value C_Small -> .1uF; footprint (none) -> Capacitor_THT:C_Rect_L4.0mm_W2.5mm_P2.50mm
- D101: renamed from D3; footprint Diode_THT:D_DO-35_SOD27_P7.62mm_Horizontal -> Diode_SMD:D_SOD-323
- D4: footprint (none) -> LED_THT:LED_D3.0mm_Horizontal_O1.27mm_Z6.0mm
- J3: renamed from U9; footprint Connector_PinHeader_2.54mm:PinHeader_1x02_P2.54mm_Vertical -> Connector_PinHeader_2.54mm:PinHeader_1x02_P2.54mm_Horizontal
- L2: footprint Inductor_THT:L_Axial_L11.0mm_D4.5mm_P15.24mm_Horizontal_Fastron_MECC -> powersupply:11R102C_Inductor
- R10, R13, R14, R15, R16, R17, R3, R6, R7, R8, R9: footprint Resistor_THT:R_Axial_DIN0207_L6.3mm_D2.5mm_P10.16mm_Horizontal -> Resistor_SMD:R_0805_2012Metric
- R18, R19, R20: footprint (none) -> Resistor_SMD:R_0805_2012Metric
- TP10: value TestPoint -> pin_2_pad
- TP11: value TestPoint -> pin_2_alt
- TP8: value TestPoint -> pin_1_alt
- TP9: value TestPoint -> pin_1_pad
- U6: footprint Package_SO:SOIC-8_3.9x4.9mm_P1.27mm -> Package_DIP:DIP-8_W7.62mm
Other:
- moved on the sheet: H1, H2, H3, H4, TP2, TP3, TP4, TP7
