File: Power_Supply/powersupply/powersupply.sch (KiCad schematic (older format))
At the start: 70 parts, among them J1 Conn_01x03, J2 USB_B_Micro, J3 1x2, J4 1x2, Q1 Q_PMOS_GDS, SW1 KMR2, U1 AZ1117E-3.3, U10 INA199, U2 ATSAMD10D13A-SS, U3 B0505S-2WR2, U5 joystick-K1-1506DN-01, U6 MC33063AP1, U7 LM358P

Commit message: renumbered
Parts:
- renumbered C5 to C1, C105 to C103, C103 to C104, C106 to C105, C104 to C106, C4 to C2, C2 to C3, C1 to C4, C3 to C5, R11 to R1, R1 to R101, R3 to R102, R101 to R103, R103 to R104, R102 to R105, R6 to R106, R7 to R107, R8 to R108, R105 to R109, R104 to R110, R20 to R111, R19 to R112, R13 to R113, R14 to R114, R16 to R115, R17 to R116, R10 to R117, R9 to R118, R15 to R119
Changed lines of the file:
@@
 $EndComp
 $Comp
-L Device:R_Small_US R13
+L Device:R_Small_US R113
 U 1 1 5D4AC3D3
 P 7750 2700
-F 0 "R13" H 7818 2746 50  0000 L CNN
+F 0 "R113" H 7818 2746 50  0000 L CNN
 F 1 "15k" H 7818 2655 50  0000 L CNN
 F 2 "Resistor_SMD:R_0805_2012Metric" H 7750 2700 50  0001 C CNN
@@
 $EndComp
 $Comp
-L Device:R_Small_US R14
+L Device:R_Small_US R114
 U 1 1 5D4AD799
 P 7750 2900
-F 0 "R14" H 7850 2950 50  0000 L CNN
+F 0 "R114" H 7850 2950 50  0000 L CNN
 F 1 "100" H 7850 2850 50  0000 L CNN
 F 2 "Resistor_SMD:R_0805_2012Metric" H 7750 2900 50  0001 C CNN
@@
 $EndComp
 $Comp
-L Device:R_Small_US R103
+L Device:R_Small_US R104
 U 1 1 5D4F946F
 P 2850 5250
-F 0 "R103" V 2645 5250 50  0000 C CNN
+F 0 "R104" V 2645 5250 50  0000 C CNN
 F 1 "1k" V 2736 5250 50  0000 C CNN
 F 2 "Resistor_SMD:R_0805_2012Metric" H 2850 5250 50  0001 C CNN
@@
 $EndComp
 $Comp
-L Device:R_Small_US R102
+L Device:R_Small_US R105
 U 1 1 5D4FAA70
 P 2600 5450
-F 0 "R102" V 2700 5450 50  0000 C CNN
+F 0 "R105" V 2700 5450 50  0000 C CNN
 F 1 "1k" V 2800 5450 50  0000 C CNN
 F 2 "Resistor_SMD:R_0805_2012Metric" H 2600 5450 50  0001 C CNN
@@
 $EndComp
 $Comp
-L Device:C_Small C103
+L Device:C_Small C104
 U 1 1 5D502474
 P 2700 5850
-F 0 "C103" H 2792 5896 50  0000 L CNN
+F 0 "C104" H 2792 5896 50  0000 L CNN
 F 1 "15uF" H 2792 5805 50  0000 L CNN
 F 2 "Capacitor_SMD:C_0805_2012Metric" H 2700 5850 50  0001 C CNN
@@
 $EndComp
 $Comp
-L Device:C_Small C105
+L Device:C_Small C103
 U 1 1 5D5092B9
 P 3150 5500
-F 0 "C105" H 3242 5546 50  0000 L CNN
+F 0 "C103" H 3242 5546 50  0000 L CNN
 F 1 "15uF" H 3242 5455 50  0000 L CNN
 F 2 "Capacitor_SMD:C_0805_2012Metric" H 3150 5500 50  0001 C CNN
@@
 $EndComp
 $Comp
-L Device:C_Small C104
+L Device:C_Small C106
 U 1 1 5D5A2D7A
 P 3300 3250
-F 0 "C104" V 3071 3250 50  0000 C CNN
+F 0 "C106" V 3071 3250 50  0000 C CNN
 F 1 "1uF" V 3162 3250 50  0000 C CNN
 F 2 "Capacitor_SMD:C_0805_2012Metric" H 3300 3250 50  0001 C CNN
@@
 	3400 3250 3550 3250
 $Comp
-L Device:R_Small_US R101
+L Device:R_Small_US R103
 U 1 1 5D4A83DB
 P 1400 3050
-F 0 "R101" H 1300 3150 50  0000 C CNN
+F 0 "R103" H 1300 3150 50  0000 C CNN
 F 1 "4.7k" H 1286 3050 50  0000 C CNN
 F 2 "Resistor_SMD:R_0805_2012Metric" H 1400 3050 50  0001 C CNN
@@
 $EndComp
 $Comp
-L Device:R_Small_US R15
+L Device:R_Small_US R119
 U 1 1 5D4B4E12
 P 9150 2800
-F 0 "R15" V 9050 2700 50  0000 L CNN
+F 0 "R119" V 9050 2700 50  0000 L CNN
 F 1 "3k" V 9050 2900 50  0000 L CNN
 F 2 "Resistor_SMD:R_0805_2012Metric" H 9150 2800 50  0001 C CNN
@@
 $EndComp
 $Comp
-L Device:R_Small_US R3
+L Device:R_Small_US R102
 U 1 1 5D459423
 P 4900 4250
-F 0 "R3" V 4695 4250 50  0000 C CNN
+F 0 "R102" V 4695 4250 50  0000 C CNN
 F 1 "180" V 4786 4250 50  0000 C CNN
 F 2 "Resistor_SMD:R_0805_2012Metric" H 4900 4250 50  0001 C CNN
@@
 Wire Wire Line
 	4800 4500 5250 4500
-$Comp
-L Device:R_Small_US R2
-U 1 1 5D45B2AA
-P 4800 4600
-F 0 "R2" H 4868 4646 50  0000 L CNN
-F 1 "0.3 1/4W" H 4868 4555 50  0000 L CNN
-F 2 "Resistor_THT:R_Axial_DIN0207_L6.3mm_D2.5mm_P10.16mm_Horizontal" H 4800 4600 50  0001 C CNN
-F 3 "~" H 4800 4600 50  0001 C CNN
-	1    4800 4600
-	1    0    0    -1
-$EndComp
 Connection ~ 4800 4500
 $Comp
-L Device:CP1_Small C1
+L Device:CP1_Small C4
 U 1 1 5D45B91C
 P 4800 4850
-F 0 "C1" H 4550 4900 50  0000 L CNN
+F 0 "C4" H 4550 4900 50  0000 L CNN
 F 1 "470uF" H 4450 4800 50  0000 L CNN
 F 2 "Capacitor_THT:CP_Radial_D8.0mm_P3.50mm" H 4800 4850 50  0001 C CNN
@@
 $EndComp
 $Comp
-L Device:R_Small_US R8
+L Device:R_Small_US R108
 U 1 1 5D46B727
 P 5500 5350
-F 0 "R8" V 5295 5350 50  0000 C CNN
+F 0 "R108" V 5295 5350 50  0000 C CNN
 F 1 "5.5k" V 5386 5350 50  0000 C CNN
 F 2 "Resistor_SMD:R_0805_2012Metric" H 5500 5350 50  0001 C CNN
@@
 	5100 5000 5250 5000
 $Comp
-L Device:CP1_Small C3
+L Device:CP1_Small C5
 U 1 1 5D46EC73
 P 6100 5450
-F 0 "C3" H 6191 5496 50  0000 L CNN
+F 0 "C5" H 6191 5496 50  0000 L CNN
 F 1 "470uF" H 6191 5405 50  0000 L CNN
 F 2 "Capacitor_THT:CP_Radial_D8.0mm_P3.50mm" H 6100 5450 50  0001 C CNN
@@
 Boost_out
 $Comp
-L Device:R_Small_US R6
+L Device:R_Small_US R106
 U 1 1 5D49225A
 P 4600 5350
-F 0 "R6" V 4395 5350 50  0000 C CNN
+F 0 "R106" V 4395 5350 50  0000 C CNN
 F 1 "3.17k" V 4486 5350 50  0000 C CNN
 F 2 "Resistor_SMD:R_0805_2012Metric" H 4600 5350 50  0001 C CNN
@@
 Connection ~ 5100 5350
 $Comp
-L Device:R_Small_US R7
+L Device:R_Small_US R107
 U 1 1 5D46A6EF
 P 5100 5450
-F 0 "R7" H 5168 5496 50  0000 L CNN
+F 0 "R107" H 5168 5496 50  0000 L CNN
 F 1 "3.6k" H 5168 5405 50  0000 L CNN
 F 2 "Resistor_SMD:R_0805_2012Metric" H 5100 5450 50  0001 C CNN
@@
 $EndComp
 $Comp
-L Device:CP1_Small C4
+L Device:CP1_Small C2
 U 1 1 5D5744DC
 P 7050 5450
-F 0 "C4" H 7141 5496 50  0000 L CNN
+F 0 "C2" H 7141 5496 50  0000 L CNN
 F 1 "100uF" H 7141 5405 50  0000 L CNN
 F 2 "Capacitor_THT:CP_Radial_D6.3mm_P2.50mm" H 7050 5450 50  0001 C CNN
@@
 $EndComp
 $Comp
-L Device:R_Small_US R9
+L Device:R_Small_US R118
 U 1 1 5D4C0D0A
 P 8650 3700
-F 0 "R9" H 8718 3746 50  0000 L CNN
+F 0 "R118" H 8718 3746 50  0000 L CNN
 F 1 "130k" H 8718 3655 50  0000 L CNN
 F 2 "Resistor_SMD:R_0805_2012Metric" H 8650 3700 50  0001 C CNN
@@
 $EndComp
 $Comp
-L Device:R_Small_US R10
+L Device:R_Small_US R117
 U 1 1 5D4C174A
 P 9100 3800
-F 0 "R10" V 9300 3800 50  0000 C CNN
+F 0 "R117" V 9300 3800 50  0000 C CNN
 F 1 "100" V 9200 3800 50  0000 C CNN
 F 2 "Resistor_SMD:R_0805_2012Metric" H 9100 3800 50  0001 C CNN
@@
 $EndComp
 $Comp
-L Device:R_Small_US R17
+L Device:R_Small_US R116
 U 1 1 5D4D044A
 P 9600 2850
-F 0 "R17" H 9668 2896 50  0000 L CNN
+F 0 "R116" H 9668 2896 50  0000 L CNN
 F 1 "2.32k" H 9668 2805 50  0000 L CNN
 F 2 "Resistor_SMD:R_0805_2012Metric" H 9600 2850 50  0001 C CNN
@@
 $EndComp
 $Comp
-L Device:R_Small_US R16
+L Device:R_Small_US R115
 U 1 1 5D4D11A0
 P 9600 3250
-F 0 "R16" H 9668 3296 50  0000 L CNN
+F 0 "R115" H 9668 3296 50  0000 L CNN
 F 1 "1k" H 9668 3205 50  0000 L CNN
 F 2 "Resistor_SMD:R_0805_2012Metric" H 9600 3250 50  0001 C CNN
@@
 	9600 3100 9600 3150
 $Comp
-L Device:R_Small_US R11
+L Device:R_Small_US R1
 U 1 1 5D4E54B6
 P 9600 3900
-F 0 "R11" H 9668 3946 50  0000 L CNN
+F 0 "R1" H 9668 3946 50  0000 L CNN
 F 1 "0.1" H 9668 3855 50  0000 L CNN
 F 2 "Resistor_THT:R_Axial_DIN0207_L6.3mm_D2.5mm_P10.16mm_Horizontal" H 9600 3900 50  0001 C CNN
@@
 	10100 2750 10700 2750
 $Comp
-L Device:CP1_Small C5
+L Device:CP1_Small C1
 U 1 1 5D53307C
 P 10100 3250
-F 0 "C5" H 10191 3296 50  0000 L CNN
+F 0 "C1" H 10191 3296 50  0000 L CNN
 F 1 "100uF" H 10191 3205 50  0000 L CNN
 F 2 "Capacitor_THT:CP_Radial_D6.3mm_P2.50mm" H 10100 3250 50  0001 C CNN
@@
 SDA
 $Comp
-L Device:R_Small_US R104
+L Device:R_Small_US R110
 U 1 1 5D5342E8
 P 10450 5200
-F 0 "R104" H 10518 5246 50  0000 L CNN
+F 0 "R110" H 10518 5246 50  0000 L CNN
 F 1 "4.7k" H 10500 5350 50  0000 L CNN
 F 2 "Resistor_SMD:R_0805_2012Metric" H 10450 5200 50  0001 C CNN
@@
 SCK
 $Comp
-L Device:R_Small_US R105
+L Device:R_Small_US R109
 U 1 1 5D5363F7
 P 10450 5600
-F 0 "R105" H 10200 5700 50  0000 L CNN
+F 0 "R109" H 10200 5700 50  0000 L CNN
 F 1 "4.7k" H 10200 5600 50  0000 L CNN
 F 2 "Resistor_SMD:R_0805_2012Metric" H 10450 5600 50  0001 C CNN
@@
 	2500 3250 2950 3250
 $Comp
-L Device:C_Small C2
+L Device:C_Small C3
 U 1 1 5D4C7F8E
 P 6700 4850
-F 0 "C2" H 6550 4900 50  0000 L CNN
+F 0 "C3" H 6550 4900 50  0000 L CNN
 F 1 "270pF" H 6300 4800 50  0000 L CNN
 F 2 "Capacitor_THT:C_Rect_L4.0mm_W2.5mm_P2.50mm" H 6700 4850 50  0001 C CNN
@@
 $EndComp
 $Comp
-L Device:R_Small_US R19
+L Device:R_Small_US R112
 U 1 1 5D61A8DD
 P 2950 4550
-F 0 "R19" H 3018 4596 50  0000 L CNN
+F 0 "R112" H 3018 4596 50  0000 L CNN
 F 1 "18.2k" H 3018 4505 50  0000 L CNN
 F 2 "Resistor_SMD:R_0805_2012Metric" H 2950 4550 50  0001 C CNN
@@
 $EndComp
 $Comp
-L Device:R_Small_US R20
+L Device:R_Small_US R111
 U 1 1 5D61B980
 P 2950 4750
-F 0 "R20" H 3018 4796 50  0000 L CNN
+F 0 "R111" H 3018 4796 50  0000 L CNN
 F 1 "4.99k" H 3018 4705 50  0000 L CNN
 F 2 "Resistor_SMD:R_0805_2012Metric" H 2950 4750 50  0001 C CNN
@@
 Connection ~ 4950 3000
 $Comp
-L Device:C_Small C106
+L Device:C_Small C105
 U 1 1 5D675D51
 P 4500 2700
-F 0 "C106" V 4271 2700 50  0000 C CNN
+F 0 "C105" V 4271 2700 50  0000 C CNN
 F 1 ".1uF" V 4362 2700 50  0000 C CNN
 F 2 "Capacitor_SMD:C_0805_2012Metric" H 4500 2700 50  0001 C CNN
@@
 	2650 1600 2950 1600
 $Comp
-L Device:R_Small_US R1
+L Device:R_Small_US R101
 U 1 1 5D5DBC0A
 P 2950 1500
-F 0 "R1" V 2750 1500 50  0000 C CNN
+F 0 "R101" V 2750 1500 50  0000 C CNN
 F 1 "150" V 2836 1500 50  0000 C CNN
 F 2 "Resistor_SMD:R_0805_2012Metric" H 2950 1500 50  0001 C CNN
@@
 $EndComp
 Connection ~ 2950 1600
-$Comp
-L Device:R_Small_US R18
-U 1 1 5D62CB9E
-P 3700 1200
-F 0 "R18" H 3768 1246 50  0000 L CNN
-F 1 "560" H 3768 1155 50  0000 L CNN
-F 2 "Resistor_THT:R_Axial_DIN0207_L6.3mm_D2.5mm_P10.16mm_Horizontal" H 3700 1200 50  0001 C CNN
-F 3 "~" H 3700 1200 50  0001 C CNN
-	1    3700 1200
-	1    0    0    -1
-$EndComp
 $Comp
 L Device:LED D4
@@
 	6100 5350 6850 5350
 Connection ~ 6850 5350
+$Comp
+L Device:R_Small_US R2
+U 1 1 5D45B2AA
+P 4800 4600
+F 0 "R2" H 4868 4646 50  0000 L CNN
+F 1 "0.3 1/4W" H 4868 4555 50  0000 L CNN
+F 2 "Resistor_THT:R_Axial_DIN0207_L6.3mm_D2.5mm_P10.16mm_Horizontal" H 4800 4600 50  0001 C CNN
+F 3 "~" H 4800 4600 50  0001 C CNN
+	1    4800 4600
+	1    0    0    -1
+$EndComp
+$Comp
+L Device:R_Small_US R18
+U 1 1 5D62CB9E
+P 3700 1200
+F 0 "R18" H 3768 1246 50  0000 L CNN
+F 1 "560" H 3768 1155 50  0000 L CNN
+F 2 "Resistor_THT:R_Axial_DIN0207_L6.3mm_D2.5mm_P10.16mm_Horizontal" H 3700 1200 50  0001 C CNN
+F 3 "~" H 3700 1200 50  0001 C CNN
+	1    3700 1200
+	1    0    0    -1
+$EndComp
 $EndSCHEMATC

Commit message: changes
Parts:
- R2: renamed from R18; value 560 -> 580
- renumbered R2 to R3
Changed lines of the file:
@@
 Connection ~ 6850 5350
 $Comp
-L Device:R_Small_US R2
+L Device:R_Small_US R3
 U 1 1 5D45B2AA
 P 4800 4600
-F 0 "R2" H 4868 4646 50  0000 L CNN
+F 0 "R3" H 4868 4646 50  0000 L CNN
 F 1 "0.3 1/4W" H 4868 4555 50  0000 L CNN
 F 2 "Resistor_THT:R_Axial_DIN0207_L6.3mm_D2.5mm_P10.16mm_Horizontal" H 4800 4600 50  0001 C CNN
@@
 $EndComp
 $Comp
-L Device:R_Small_US R18
+L Device:R_Small_US R2
 U 1 1 5D62CB9E
 P 3700 1200
-F 0 "R18" H 3768 1246 50  0000 L CNN
-F 1 "560" H 3768 1155 50  0000 L CNN
+F 0 "R2" H 3768 1246 50  0000 L CNN
+F 1 "580" H 3768 1155 50  0000 L CNN
 F 2 "Resistor_THT:R_Axial_DIN0207_L6.3mm_D2.5mm_P10.16mm_Horizontal" H 3700 1200 50  0001 C CNN
 F 3 "~" H 3700 1200 50  0001 C CNN

Commit message: finished
Parts:
- D1: renamed from D4; footprint LED_THT:LED_D3.0mm -> LED_THT:LED_D5.0mm
- TP4: renamed from TP6; value Boost_ctrl -> Boost_c
- renumbered D1 to D2, D2 to D3, TP3 to TP1, TP4 to TP3, TP1 to TP6, U3 to U1, U1 to U101, U2 to U102, U6 to U2, U7 to U3, U5 to U4
Changed lines of the file:
@@
 NoConn ~ 1200 1550
 $Comp
-L powersupply:RFM-0505S U3
+L powersupply:RFM-0505S U1
 U 1 1 5D303F43
 P 2400 850
-F 0 "U3" H 2400 775 50  0000 C CNN
+F 0 "U1" H 2400 775 50  0000 C CNN
 F 1 "B0505S-2WR2" H 2400 684 50  0000 C CNN
 F 2 "powersupply:B0505S-2WR2-Isolator" H 2400 850 50  0001 C CNN
@@
 Connection ~ 6200 1150
 $Comp
-L powersupply:ATSAMD10D13A-SS U2
+L powersupply:ATSAMD10D13A-SS U102
 U 1 1 5D47B7D4
 P 2100 3450
-F 0 "U2" H 1150 3150 50  0000 C CNN
+F 0 "U102" H 1150 3150 50  0000 C CNN
 F 1 "ATSAMD10D13A-SS" H 1100 3000 50  0000 C CNN
 F 2 "Package_SO:SOIC-20W_7.5x12.8mm_P1.27mm" H 2100 2300 50  0001 C CNN
@@
 $EndComp
 $Comp
-L powersupply:LM358P U7
+L powersupply:LM358P U3
 U 1 1 5D4A8FA5
 P 8600 2500
-F 0 "U7" H 8575 2615 50  0000 C CNN
+F 0 "U3" H 8575 2615 50  0000 C CNN
 F 1 "LM358P" H 8575 2524 50  0000 C CNN
 F 2 "Package_DIP:DIP-8_W7.62mm" H 8600 2500 50  0001 C CNN
@@
 	3150 5250 3150 5400
 $Comp
-L Regulator_Linear:AZ1117-3.3 U1
+L Regulator_Linear:AZ1117-3.3 U101
 U 1 1 5D489A61
 P 5600 1150
-F 0 "U1" H 5600 1392 50  0000 C CNN
+F 0 "U101" H 5600 1392 50  0000 C CNN
 F 1 "AZ1117E-3.3" H 5600 1301 50  0000 C CNN
 F 2 "Package_TO_SOT_SMD:SOT-223-3_TabPin2" H 5600 1400 50  0001 C CIN
@@
 SWDIO
 $Comp
-L powersupply:joystick-K1-1506DN-01 U5
+L powersupply:joystick-K1-1506DN-01 U4
 U 1 1 5D4C0110
 P 5750 6400
-F 0 "U5" H 5750 6400 50  0000 C CNN
+F 0 "U4" H 5750 6400 50  0000 C CNN
 F 1 "joystick-K1-1506DN-01" H 5800 6300 50  0000 C CNN
 F 2 "powersupply:K1-1506DN-01_joystick" H 5750 6400 50  0001 C CNN
@@
 $EndComp
 $Comp
-L powersupply:MC33063AP1 U6
+L powersupply:MC33063AP1 U2
 U 1 1 5D455E56
 P 5750 4100
-F 0 "U6" H 5750 4215 50  0000 C CNN
+F 0 "U2" H 5750 4215 50  0000 C CNN
 F 1 "MC33063AP1" H 5750 4124 50  0000 C CNN
 F 2 "Package_DIP:DIP-8_W7.62mm" H 5750 4100 50  0001 C CNN
@@
 $EndComp
 $Comp
-L Device:D_Schottky_Small D2
+L Device:D_Schottky_Small D3
 U 1 1 5D4E566E
 P 8600 2250
-F 0 "D2" H 8600 2045 50  0000 C CNN
+F 0 "D3" H 8600 2045 50  0000 C CNN
 F 1 "1N5819" H 8600 2136 50  0000 C CNN
 F 2 "Diode_THT:D_DO-41_SOD81_P7.62mm_Horizontal" V 8600 2250 50  0001 C CNN
@@
 $EndComp
 $Comp
-L Device:D_Schottky_Small D1
+L Device:D_Schottky_Small D2
 U 1 1 5D4EED9B
 P 6850 4550
-F 0 "D1" V 6896 4482 50  0000 R CNN
+F 0 "D2" V 6896 4482 50  0000 R CNN
 F 1 "1N5819" V 6805 4482 50  0000 R CNN
 F 2 "Diode_THT:D_DO-41_SOD81_P7.62mm_Horizontal" V 6850 4550 50  0001 C CNN
@@
 $EndComp
 $Comp
-L Connector:TestPoint TP3
+L Connector:TestPoint TP1
 U 1 1 5D4B6929
 P 1250 6900
-F 0 "TP3" H 1192 6926 50  0000 R CNN
+F 0 "TP1" H 1192 6926 50  0000 R CNN
 F 1 "+3.3" H 1192 7017 50  0000 R CNN
 F 2 "Connector_PinHeader_1.00mm:PinHeader_1x01_P1.00mm_Vertical" H 1450 6900 50  0001 C CNN
@@
 $EndComp
 $Comp
-L Connector:TestPoint TP1
+L Connector:TestPoint TP6
 U 1 1 5D4B7B24
 P 4300 7200
-F 0 "TP1" H 4358 7318 50  0000 L CNN
+F 0 "TP6" H 4358 7318 50  0000 L CNN
 F 1 "Boost_out" H 4358 7227 50  0000 L CNN
 F 2 "Connector_PinHeader_1.00mm:PinHeader_1x01_P1.00mm_Vertical" H 4500 7200 50  0001 C CNN
@@
 $EndComp
 $Comp
-L Connector:TestPoint TP4
+L Connector:TestPoint TP3
 U 1 1 5D4B85BC
 P 3250 6950
-F 0 "TP4" H 3308 7068 50  0000 L CNN
+F 0 "TP3" H 3308 7068 50  0000 L CNN
 F 1 "Current_limit" H 3308 6977 50  0000 L CNN
 F 2 "Connector_PinHeader_1.00mm:PinHeader_1x01_P1.00mm_Vertical" H 3450 6950 50  0001 C CNN
@@
 Voltage_limit_divider
 $Comp
-L Connector:TestPoint TP6
+L Connector:TestPoint TP4
 U 1 1 5D4BF42E
 P 4300 6950
-F 0 "TP6" H 4358 7068 50  0000 L CNN
-F 1 "Boost_ctrl" H 4358 6977 50  0000 L CNN
+F 0 "TP4" H 4358 7068 50  0000 L CNN
+F 1 "Boost_c" H 4358 6977 50  0000 L CNN
 F 2 "Connector_PinHeader_1.00mm:PinHeader_1x01_P1.00mm_Vertical" H 4500 6950 50  0001 C CNN
 F 3 "~" H 4500 6950 50  0001 C CNN
@@
 Connection ~ 2950 1600
 $Comp
-L Device:LED D4
+L Device:LED D1
 U 1 1 5D62BB53
 P 3700 1450
-F 0 "D4" V 3739 1332 50  0000 R CNN
+F 0 "D1" V 3739 1332 50  0000 R CNN
 F 1 "C503B 2.1V" V 3648 1332 50  0000 R CNN
-F 2 "LED_THT:LED_D3.0mm" H 3700 1450 50  0001 C CNN
+F 2 "LED_THT:LED_D5.0mm" H 3700 1450 50  0001 C CNN
 F 3 "~" H 3700 1450 50  0001 C CNN
 	1    3700 1450
