File: Power_Supply/powersupply/powersupply.kicad_pcb (KiCad board)
At the start: 2 copper layers, 60.8 x 63.3 mm, 70 parts, among them J1 Conn_01x03, J2 USB_B_Micro, J3 1x2, J4 1x2, Q1 Q_PMOS_GDS, SW1 KMR2, U1 AZ1117E-3.3, U10 INA199, U2 ATSAMD10D13A-SS, U3 B0505S-2WR2, U5 joystick-K1-1506DN-01, U6 MC33063AP1, U7 LM358P

Commit message: changes
Routing:
- net /V_negative_out: track 93.8 -> 94.6 mm
- net +3V3: track 161.1 -> 161.8 mm

Commit message: renumbered
Parts:
- TP13: value TestPoint -> pin_2_pad_alt
- renumbered C5 to C1, C105 to C103, C103 to C104, C106 to C105, C104 to C106, C4 to C2, C2 to C3, C1 to C4, C3 to C5, R11 to R1, R1 to R101, R3 to R102, R101 to R103, R103 to R104, R102 to R105, R6 to R106, R7 to R107, R8 to R108, R105 to R109, R104 to R110, R20 to R111, R19 to R112, R13 to R113, R14 to R114, R16 to R115, R17 to R116, R10 to R117, R9 to R118, R15 to R119
Connections:
- net Net-(J2-Pad1) renamed /USB_5V
- net Net-(J2-Pad5) renamed /USB_GND

Commit message: changes
Parts:
- R2: renamed from R18; value 560 -> 580
- renumbered R2 to R3

Commit message: finished
Parts:
- D1: renamed from D4; footprint LED_THT:LED_D3.0mm -> LED_THT:LED_D5.0mm
- TP4: renamed from TP6; value Boost_ctrl -> Boost_c
- moved D1 0.21 mm to (41.0, 47.4)
- renumbered D1 to D2, D2 to D3, TP3 to TP1, TP4 to TP3, TP1 to TP6, U3 to U1, U1 to U101, U2 to U102, U6 to U2, U7 to U3, U5 to U4
Other:
- board text added: "+5V Iso"
- board text added: "Boost c"
- board text removed: "+5V"
- board text removed: "Boost"

Commit message: little layout changes
Other:
- board text added: "Power Supply"
Changed lines of the file:
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@@
   (general
     (thickness 1.6)
-    (drawings 26)
+    (drawings 25)
     (tracks 525)
     (zones 0)
@@
   (page A4)
   (layers
-    (0 F.Cu signal hide)
-    (31 B.Cu signal hide)
+    (0 F.Cu signal)
+    (31 B.Cu signal)
     (32 B.Adhes user)
     (33 F.Adhes user)
@@
     )
   )
+  (gr_line (start 59.15 34.58) (end 59.15 35) (layer B.SilkS) (width 0.12))
+  (gr_line (start 59.15 35.3) (end 59.15 35.72) (layer B.SilkS) (width 0.12))
+  (gr_line (start 59.15 33.15) (end 59.15 33.57) (layer B.SilkS) (width 0.12))
+  (gr_line (start 59.15 33.88) (end 59.15 34.3) (layer B.SilkS) (width 0.12))
+  (gr_line (start 55.91 35.29) (end 55.91 35.71) (layer B.SilkS) (width 0.12))
+  (gr_line (start 55.91 34.57) (end 55.91 34.99) (layer B.SilkS) (width 0.12))
+  (gr_line (start 55.91 33.87) (end 55.91 34.29) (layer B.SilkS) (width 0.12))
+  (gr_line (start 55.91 33.14) (end 55.91 33.56) (layer B.SilkS) (width 0.12))
+  (gr_text "Power Supply" (at 59.53 57.06) (layer B.SilkS)
+    (effects (font (size 5 5) (thickness 0.5)) (justify mirror))
+  )
   (gr_arc (start 32.27 31.55) (end 32.27 28.1) (angle -90) (layer Edge.Cuts) (width 0.05))
   (gr_arc (start 32.27 87.95) (end 28.82 87.95) (angle -90) (layer Edge.Cuts) (width 0.05))
@@
     (effects (font (size 1 1) (thickness 0.25)) (justify right))
   )
-  (gr_line (start 59.16 34.95) (end 59.16 35.23) (layer F.SilkS) (width 0.12))
-  (gr_line (start 59.16 33.13) (end 59.16 33.41) (layer F.SilkS) (width 0.12))
-  (gr_line (start 59.16 34.32) (end 59.16 34.6) (layer F.SilkS) (width 0.12))
-  (gr_line (start 59.16 33.73) (end 59.16 34.01) (layer F.SilkS) (width 0.12))
-  (gr_line (start 59.16 35.57) (end 59.16 35.85) (layer F.SilkS) (width 0.12))
-  (gr_line (start 55.89 34.92) (end 55.89 35.2) (layer F.SilkS) (width 0.12))
-  (gr_line (start 55.89 33.1) (end 55.89 33.38) (layer F.SilkS) (width 0.12))
-  (gr_line (start 55.89 34.29) (end 55.89 34.57) (layer F.SilkS) (width 0.12))
-  (gr_line (start 55.89 33.7) (end 55.89 33.98) (layer F.SilkS) (width 0.12))
-  (gr_line (start 55.89 35.54) (end 55.89 35.82) (layer F.SilkS) (width 0.12))
   (gr_arc (start 86.12 31.54) (end 89.57 31.54) (angle -90) (layer Edge.Cuts) (width 0.05))
   (gr_line (start 32.27 28.1) (end 86.12 28.1) (layer Edge.Cuts) (width 0.05))
@@
   (segment (start 77.015 49.36) (end 76.385 48.73) (width 0.25) (layer F.Cu) (net 8))
   (segment (start 77.69 49.36) (end 77.015 49.36) (width 0.25) (layer F.Cu) (net 8))
+  (segment (start 49.77 44.125) (end 49.77 39.19) (width 0.25) (layer F.Cu) (net 9))
+  (segment (start 46.245 47.65) (end 49.77 44.125) (width 0.25) (layer F.Cu) (net 9))
+  (segment (start 43.935 47.65) (end 46.245 47.65) (width 0.25) (layer F.Cu) (net 9))
   (segment (start 53.88 69.38) (end 53.88 70.74) (width 0.25) (layer F.Cu) (net 10))
   (segment (start 49.6 65.1) (end 53.88 69.38) (width 0.25) (layer F.Cu) (net 10))
   (segment (start 44.24 70.46) (end 44.24 71.3) (width 0.25) (layer F.Cu) (net 10))
   (segment (start 49.6 65.1) (end 44.24 70.46) (width 0.25) (layer F.Cu) (net 10))
-  (segment (start 82.49 61.7) (end 82.49 64.87) (width 0.25) (layer F.Cu) (net 40))
-  (segment (start 81.22 70.97) (end 81.740001 71.490001) (width 0.25) (layer F.Cu) (net 40))
-  (segment (start 82.49 64.87) (end 81.22 66.14) (width 0.25) (layer F.Cu) (net 40))
-  (segment (start 81.740001 71.490001) (end 82.84 72.59) (width 0.25) (layer F.Cu) (net 40))
-  (segment (start 81.22 66.14) (end 81.22 70.97) (width 0.25) (layer F.Cu) (net 40))
-  (segment (start 76.4925 79.4775) (end 74.55 79.4775) (width 0.25) (layer F.Cu) (net 41))
-  (segment (start 77.21 78.76) (end 76.4925 79.4775) (width 0.25) (layer F.Cu) (net 41))
-  (segment (start 79.87 78.76) (end 77.21 78.76) (width 0.25) (layer F.Cu) (net 41))
-  (segment (start 74.4775 79.55) (end 74.55 79.4775) (width 0.25) (layer F.Cu) (net 41))
-  (segment (start 73.8 79.55) (end 74.4775 79.55) (width 0.25) (layer F.Cu) (net 41))
-  (segment (start 73 78.75) (end 73.8 79.55) (width 0.25) (layer F.Cu) (net 41))
-  (segment (start 75.22 74.58) (end 73 76.8) (width 0.25) (layer F.Cu) (net 41))
-  (segment (start 73 76.8) (end 73 78.75) (width 0.25) (layer F.Cu) (net 41))
-  (segment (start 75.22 72.59) (end 75.22 74.58) (width 0.25) (layer F.Cu) (net 41))
   (segment (start 58.3 40.37) (end 61.72 40.37) (width 0.25) (layer F.Cu) (net 11))
   (segment (start 48.66 37.56) (end 55.49 37.56) (width 0.25) (layer F.Cu) (net 11))
@@
   (segment (start 84.3425 58.4) (end 84.7 58.7575) (width 0.25) (layer F.Cu) (net 29))
   (segment (start 82.55 58.4) (end 84.3425 58.4) (width 0.25) (layer F.Cu) (net 29))
-  (segment (start 49.77 44.125) (end 49.77 39.19) (width 0.25) (layer F.Cu) (net 9))
-  (segment (start 46.245 47.65) (end 49.77 44.125) (width 0.25) (layer F.Cu) (net 9))
-  (segment (start 43.935 47.65) (end 46.245 47.65) (width 0.25) (layer F.Cu) (net 9))
   (segment (start 38.62 29.725) (end 44.42 29.725) (width 0.25) (layer F.Cu) (net 30))
   (segment (start 44.42 32.025) (end 44.02 32.425) (width 0.25) (layer F.Cu) (net 30))
@@
   (segment (start 77.41 74.7425) (end 74.55 77.6025) (width 0.25) (layer F.Cu) (net 39))
   (segment (start 77.41 69.32) (end 77.41 74.7425) (width 0.25) (layer F.Cu) (net 39))
+  (segment (start 82.49 61.7) (end 82.49 64.87) (width 0.25) (layer F.Cu) (net 40))
+  (segment (start 81.22 70.97) (end 81.740001 71.490001) (width 0.25) (layer F.Cu) (net 40))
+  (segment (start 82.49 64.87) (end 81.22 66.14) (width 0.25) (layer F.Cu) (net 40))
+  (segment (start 81.740001 71.490001) (end 82.84 72.59) (width 0.25) (layer F.Cu) (net 40))
+  (segment (start 81.22 66.14) (end 81.22 70.97) (width 0.25) (layer F.Cu) (net 40))
+  (segment (start 76.4925 79.4775) (end 74.55 79.4775) (width 0.25) (layer F.Cu) (net 41))
+  (segment (start 77.21 78.76) (end 76.4925 79.4775) (width 0.25) (layer F.Cu) (net 41))
+  (segment (start 79.87 78.76) (end 77.21 78.76) (width 0.25) (layer F.Cu) (net 41))
+  (segment (start 74.4775 79.55) (end 74.55 79.4775) (width 0.25) (layer F.Cu) (net 41))
+  (segment (start 73.8 79.55) (end 74.4775 79.55) (width 0.25) (layer F.Cu) (net 41))
+  (segment (start 73 78.75) (end 73.8 79.55) (width 0.25) (layer F.Cu) (net 41))
+  (segment (start 75.22 74.58) (end 73 76.8) (width 0.25) (layer F.Cu) (net 41))
+  (segment (start 73 76.8) (end 73 78.75) (width 0.25) (layer F.Cu) (net 41))
+  (segment (start 75.22 72.59) (end 75.22 74.58) (width 0.25) (layer F.Cu) (net 41))
   (zone (net 1) (net_name GND) (layer B.Cu) (hatch edge 0.508)
     (connect_pads (clearance 0.508))

Commit message: things
Parts:
- removed C106: 1uF, Capacitor_SMD:C_0805_2012Metric
- R101: footprint Resistor_SMD:R_0805_2012Metric -> Resistor_SMD:R_1206_3216Metric
- R103, R109, R110: value 4.7k -> 4.99k
- moved R118 39.4 mm to (44.2, 78.3), turned to 0 degrees
- moved C105 39.4 mm to (36.6, 81.6), turned to 90 degrees
- moved U102 36.9 mm to (32.4, 81.5), turned to 180 degrees
- moved R117 32.7 mm to (49.0, 78.3), turned to 0 degrees
- moved C5 22.0 mm to (46.6, 70.6)
- moved R108 21.4 mm to (65.2, 69.4), turned to 270 degrees
- moved R106 20.3 mm to (71.2, 69.4), turned to 270 degrees
- moved R107 19.5 mm to (68.2, 69.4), turned to 270 degrees
- moved C2 15.9 mm to (66.6, 76.4)
- moved TP2 13.3 mm to (21.5, 76.3)
- moved TP1 12.9 mm to (20.8, 80.7)
- moved D2 11.6 mm to (40.2, 68.0)
- moved R1 11.0 mm to (40.0, 81.5)
- moved C3 7.63 mm to (53.1, 74.3)
- moved C1 2.79 mm to (41.3, 87.0)
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- renumbered U4 to SW2, U10 to U102, U102 to U103
Connections:
- U103 pad 19: +3V3 -> Net-(U103-Pad19)
Routing:
- net /V_current_amplified: track 11.8 -> 62.8 mm, vias 0 -> 2
- net /V_negative_out: track 94.6 -> 51.5 mm, vias 2 -> 0
- net Net-(R106-Pad2): track 52.2 -> 13.7 mm
- net Net-(R117-Pad1): track 6.58 -> 43.2 mm
- net Net-(C5-Pad1): track 66.9 -> 31.1 mm
- net +3V3: track 161.8 -> 137.8 mm, vias 2 -> 4
- net /V_boost_ctrl: track 19.4 -> 40.5 mm
- net /Boost_out: track 60.4 -> 52.4 mm, vias 0 -> 1
- net Net-(L1-Pad1): track 24.2 -> 31.7 mm
- net Net-(D2-Pad2): track 15.8 -> 22.4 mm
- net Net-(C3-Pad1): track 4.20 -> 7.38 mm
- net +5V: track 116.8 -> 119.9 mm
- net GND: track 45.4 -> 42.5 mm
- net Net-(R102-Pad1): track 11.2 -> 13.3 mm
- net /V_lin_ctrl: track 54.3 -> 52.2 mm, vias 4 -> 3
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Other:
- board text added: "C"
- board text added: "D"

Commit message: changes
Parts:
- moved R2 1.84 mm to (49.0, 51.0)
Routing:
- net /V_lin_ctrl: track 52.2 -> 57.4 mm
- net Net-(D1-Pad2): track 12.2 -> 8.80 mm
- net +3V3: track 137.8 -> 140.0 mm
- net +5V: track 119.9 -> 117.9 mm
- net /V_curr_lim: track 26.1 -> 24.3 mm
- net /V_current_amplified: track 62.8 -> 61.2 mm

Commit message: finished the layout
Parts:
- moved TP1 35.5 mm to (33.9, 43.1)
- moved TP2 11.7 mm to (32.2, 78.0)
- moved R101 4.89 mm to (36.1, 38.2)
- moved D101 4.71 mm to (32.0, 38.2)
- renumbered TP2 to TP1, TP1 to TP2, U102 to U10, U103 to U102
Routing:
- net +5V: track 117.9 -> 123.5 mm
- net +3V3: track 140.0 -> 142.0 mm
- net /USB_GND: track 35.3 -> 37.1 mm
- net GND: track 42.5 -> 43.4 mm
- net /SWCLK: track 30.1 -> 29.3 mm
- net /USB_5V: track 29.1 -> 29.9 mm
- net /V_current_amplified: track 61.2 -> 61.9 mm
Other:
- outline, holes or cut-outs redrawn
