File: Power_Supply/powersupply.kicad_pcb (KiCad board)
At the start: 2 copper layers, 60.8 x 63.3 mm, 80 parts, among them J101 USB_B_Micro, J2 1x2, J3 1x2, J4 Conn_01x03_Male, Q1 IRF9Z24NPBF, SW1 KMR2, SW2 joystick-K1-1506DN-01, U101 AZ1117E-3.3, U102 INA199, U103 STM32F103C8T6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

Commit message: labels
Other:
- board text added: "D C"
Changed lines of the file:
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@@
   (general
     (thickness 1.6)
-    (drawings 29)
+    (drawings 30)
     (tracks 619)
     (zones 0)
@@
     )
   )
+  (gr_text "D   C" (at 41.148 36.068) (layer F.SilkS)
+    (effects (font (size 1.5 1.5) (thickness 0.3)))
+  )
   (gr_text "V Boost\nCtrl" (at 75.47 51.7) (layer F.SilkS)

Commit message: layout changes
Parts:
- D102: renamed from D1; footprint LED_THT:LED_D3.0mm -> LED_SMD:LED_0603_1608Metric_Pad1.05x0.95mm_HandSolder
- R123: renamed from R2; footprint Resistor_THT:R_Axial_DIN0207_L6.3mm_D2.5mm_P10.16mm_Horizontal -> Resistor_SMD:R_0805_2012Metric
- moved U101 25.4 mm to (36.1, 45.5), turned to 0 degrees
- moved C105 24.7 mm to (32.0, 57.3), turned to 270 degrees
- moved U102 24.4 mm to (36.2, 57.4), turned to 0 degrees
- moved TP2 11.9 mm to (35.9, 66.8), turned to 180 degrees
- moved D102 9.07 mm to (43.2, 38.6), turned to 180 degrees
- moved C108 6.80 mm to (49.5, 38.6), turned to 180 degrees
- moved C107 6.58 mm to (45.0, 41.9), turned to 180 degrees
- moved D2 6.38 mm to (40.6, 70.9)
- moved TP1 5.03 mm to (34.0, 38.4)
- moved R102 3.41 mm to (40.6, 57.9)
- moved R123 3.11 mm to (38.4, 38.6)
- moved Y101 2.18 mm to (53.6, 40.4), turned to 270 degrees
- moved C109 1.91 mm to (49.5, 41.9)
Routing:
- net /V_current_amplified: track 65.3 -> 29.9 mm
- net +5V: track 145.8 -> 124.4 mm
- net /V_negative_out: track 59.2 -> 80.4 mm
- net Net-(C109-Pad1): track 17.2 -> 9.41 mm
- net Net-(D102-Pad2): track 9.46 -> 3.01 mm
- net Net-(L1-Pad1): track 26.2 -> 32.3 mm
- net Net-(R102-Pad1): track 14.2 -> 17.6 mm
- net Net-(C5-Pad1): track 35.3 -> 32.1 mm
- net GND: track 83.8 -> 87.0 mm, vias 24 -> 26
- net Net-(D2-Pad2): track 26.3 -> 23.5 mm
- net Net-(C108-Pad1): track 9.14 -> 10.5 mm
- net +3V3: track 158.7 -> 158.9 mm, vias 6 -> 5
Other:
- board text added: "+5V"
- board text removed: "+5V I"
- board text removed: "- - cut iso"

Commit message: more layout
Routing:
- net GND: track 87.0 -> 85.1 mm, vias 26 -> 25
- net +3V3: track 158.9 -> 158.1 mm
- net /V_curr_lim: vias 2 -> 0
Changed lines of the file:
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@@
     (thickness 1.6)
     (drawings 28)
-    (tracks 599)
+    (tracks 596)
     (zones 0)
     (modules 80)
@@
     (tags resistor)
     (attr smd)
-    (fp_text reference R122 (at 0 -1.65 90) (layer F.SilkS)
+    (fp_text reference R122 (at -0.058 -3.03 180) (layer F.SilkS)
       (effects (font (size 1 1) (thickness 0.15)))
     )
@@
   (segment (start 46.616239 56.813761) (end 45.665467 55.862989) (width 0.4) (layer F.Cu) (net 1))
   (segment (start 61.53 63.33) (end 59.161739 60.961739) (width 0.4) (layer F.Cu) (net 1))
-  (segment (start 32.918 48.766) (end 32.918 47.766) (width 0.25) (layer F.Cu) (net 1) (status 1000000))
-  (segment (start 35.2645 51.1125) (end 32.918 48.766) (width 0.25) (layer F.Cu) (net 1) (status 1000000))
+  (segment (start 32.918 48.766) (end 32.918 47.766) (width 0.25) (layer F.Cu) (net 1))
+  (segment (start 35.2645 51.1125) (end 32.918 48.766) (width 0.25) (layer F.Cu) (net 1))
   (via (at 39.118653 55.375) (size 0.8) (drill 0.4) (layers F.Cu B.Cu) (net 1))
   (segment (start 39.606642 55.862989) (end 39.118653 55.375) (width 0.25) (layer F.Cu) (net 1))
@@
   (segment (start 59.74 34.45) (end 59.76 34.43) (width 0.25) (layer B.Cu) (net 5))
   (segment (start 58.31 34.45) (end 59.74 34.45) (width 0.25) (layer B.Cu) (net 5))
-  (segment (start 66.715002 44.881998) (end 66.033004 44.2) (width 0.25) (layer F.Cu) (net 5))
-  (segment (start 66.715002 46.857498) (end 66.715002 44.881998) (width 0.25) (layer F.Cu) (net 5))
-  (segment (start 66.46 47.1125) (end 66.715002 46.857498) (width 0.25) (layer F.Cu) (net 5))
   (segment (start 68.175 47.1125) (end 68.4925 47.43) (width 0.25) (layer F.Cu) (net 5))
   (segment (start 66.46 47.1125) (end 68.175 47.1125) (width 0.25) (layer F.Cu) (net 5))
@@
   (segment (start 35.892 64.086) (end 35.892 66.75) (width 0.25) (layer B.Cu) (net 5))
   (segment (start 35.306 63.5) (end 35.892 64.086) (width 0.25) (layer B.Cu) (net 5))
+  (segment (start 66.41001 46.259308) (end 66.41001 44.577006) (width 0.25) (layer F.Cu) (net 5))
+  (segment (start 66.43501 46.284308) (end 66.41001 46.259308) (width 0.25) (layer F.Cu) (net 5))
+  (segment (start 66.43501 47.08751) (end 66.43501 46.284308) (width 0.25) (layer F.Cu) (net 5))
+  (segment (start 66.46 47.1125) (end 66.43501 47.08751) (width 0.25) (layer F.Cu) (net 5))
   (segment (start 57.96 50.8875) (end 58.5 50.8875) (width 0.25) (layer F.Cu) (net 6))
   (segment (start 56.3875 52.46) (end 57.96 50.8875) (width 0.25) (layer F.Cu) (net 6))
@@
   (segment (start 58.5 50.8875) (end 57.89 51.4975) (width 0.25) (layer F.Cu) (net 6))
   (segment (start 72.9875 52.5625) (end 72.9875 52.5625) (width 0.25) (layer F.Cu) (net 6))
-  (via (at 72.9875 52.5625) (size 0.8) (drill 0.4) (layers F.Cu B.Cu) (net 6))
   (segment (start 72.9875 52.5625) (end 76.86 52.5625) (width 0.25) (layer F.Cu) (net 6))
-  (via (at 72.9875 52.5625) (size 0.8) (drill 0.4) (layers F.Cu B.Cu) (net 6))
   (segment (start 54.345 49.0425) (end 54.5025 49.2) (width 0.25) (layer F.Cu) (net 7))
   (segment (start 52.41 49.0425) (end 54.345 49.0425) (width 0.25) (layer F.Cu) (net 7))
@@
   (segment (start 55.35 62.23) (end 56.45 63.33) (width 0.25) (layer F.Cu) (net 23))
   (segment (start 41.5775 57.912) (end 43.19053 59.52503) (width 0.25) (layer F.Cu) (net 23))
-  (segment (start 60.5625 47.51) (end 60.5625 50.64) (width 0.25) (layer F.Cu) (net 24))
-  (segment (start 60.96 47.1125) (end 60.5625 47.51) (width 0.25) (layer F.Cu) (net 24))
+  (segment (start 60.5625 49.1655) (end 60.5625 50.64) (width 0.25) (layer F.Cu) (net 24))
+  (segment (start 60.96 48.768) (end 60.5625 49.1655) (width 0.25) (layer F.Cu) (net 24))
+  (segment (start 60.96 47.1125) (end 60.96 48.768) (width 0.25) (layer F.Cu) (net 24))
   (segment (start 71.1 69.6125) (end 71.15 69.6625) (width 0.25) (layer F.Cu) (net 25))
   (segment (start 67.95 69.6125) (end 71.1 69.6125) (width 0.25) (layer F.Cu) (net 25))
@@
   (segment (start 69.6375 71.5375) (end 69.6 71.5) (width 0.25) (layer F.Cu) (net 58))
   (segment (start 71.15 71.5375) (end 69.6375 71.5375) (width 0.25) (layer F.Cu) (net 58))
-  (via (at 65.95 45.23) (size 0.8) (drill 0.4) (layers F.Cu B.Cu) (net 58))
-  (segment (start 65.96 47.1125) (end 65.96 45.24) (width 0.25) (layer F.Cu) (net 58))
-  (segment (start 65.96 45.24) (end 65.95 45.23) (width 0.25) (layer F.Cu) (net 58))
   (via (at 62.22 40.53) (size 0.8) (drill 0.4) (layers F.Cu B.Cu) (net 58))
   (segment (start 61.46 38.7875) (end 61.46 39.77) (width 0.25) (layer F.Cu) (net 58))
@@
   (segment (start 61.46 36.8475) (end 61.46 38.7875) (width 0.25) (layer F.Cu) (net 58))
   (segment (start 61.0225 36.41) (end 61.46 36.8475) (width 0.25) (layer F.Cu) (net 58))
-  (via (at 61.92 32.73499) (size 0.8) (drill 0.4) (layers F.Cu B.Cu) (net 58))
-  (segment (start 61.48 34.43) (end 61.48 33.17499) (width 0.25) (layer B.Cu) (net 58))
-  (segment (start 61.48 33.17499) (end 61.520001 33.134989) (width 0.25) (layer B.Cu) (net 58))
-  (segment (start 61.520001 33.134989) (end 61.92 32.73499) (width 0.25) (layer B.Cu) (net 58))
   (segment (start 72.4275 39.95) (end 73.744979 39.95) (width 0.25) (layer F.Cu) (net 58))
   (via (at 73.744979 39.95) (size 0.8) (drill 0.4) (layers F.Cu B.Cu) (net 58))
@@
   (segment (start 30.3705 58.2755) (end 30.226 58.42) (width 0.25) (layer F.Cu) (net 58))
   (via (at 38.03499 57.33299) (size 0.8) (drill 0.4) (layers F.Cu B.Cu) (net 58))
-  (segment (start 40.45 52.9875) (end 41.5825 52.9875) (width 0.25) (layer F.Cu) (net 58) (status 1000000))
-  (segment (start 41.5825 52.9875) (end 42.42 52.15) (width 0.25) (layer F.Cu) (net 58) (status 1000000))
-  (segment (start 44.52 51.1125) (end 43.4575 51.1125) (width 0.25) (layer F.Cu) (net 58) (status 1000000))
-  (segment (start 43.4575 51.1125) (end 42.42 52.15) (width 0.25) (layer F.Cu) (net 58) (status 1000000))
-  (via (at 42.42 52.15) (size 0.8) (drill 0.4) (layers F.Cu B.Cu) (net 58) (status 1000000))
+  (segment (start 40.45 52.9875) (end 41.5825 52.9875) (width 0.25) (layer F.Cu) (net 58))
+  (segment (start 41.5825 52.9875) (end 42.42 52.15) (width 0.25) (layer F.Cu) (net 58))
+  (segment (start 44.52 51.1125) (end 43.4575 51.1125) (width 0.25) (layer F.Cu) (net 58))
+  (segment (start 43.4575 51.1125) (end 42.42 52.15) (width 0.25) (layer F.Cu) (net 58))
+  (via (at 42.42 52.15) (size 0.8) (drill 0.4) (layers F.Cu B.Cu) (net 58))
+  (segment (start 65.931999 45.865999) (end 65.532 45.466) (width 0.25) (layer F.Cu) (net 58))
+  (via (at 65.532 45.466) (size 0.8) (drill 0.4) (layers F.Cu B.Cu) (net 58))
+  (segment (start 65.96 47.1125) (end 65.96 45.894) (width 0.25) (layer F.Cu) (net 58))
+  (segment (start 65.96 45.894) (end 65.931999 45.865999) (width 0.25) (layer F.Cu) (net 58))
   (segment (start 56.23 46.9775) (end 56.28 47.0275) (width 0.25) (layer F.Cu) (net 59))
   (segment (start 53 46.9775) (end 56.23 46.9775) (width 0.25) (layer F.Cu) (net 59))

Commit message: logo
Parts:
- added G***: LOGO, powersupply:Logo, B.Cu at (59.4, 65.5)

Commit message: layout
Parts:
- removed G***: LOGO, powersupply:Logo
- removed TP10: pad_2, powersupply:pads
- removed TP11: pin_2_alt, powersupply:pads
- removed TP12: Pad1_default, powersupply:pads
- removed TP13: pin_2_pad_alt, powersupply:pads
- removed TP8: pin_1_alt, powersupply:pads
- removed TP9: pad_1, powersupply:pads
- added J103: Default_Jumper, powersupply:Default_Jumper, B.Cu at (58.2, 34.3)
- added J104: Default_Jumper, powersupply:Default_Jumper, B.Cu at (53.6, 34.3)
- D101: renamed from D102; footprint LED_SMD:LED_0603_1608Metric_Pad1.05x0.95mm_HandSolder -> LED_SMD:LED_0805_2012Metric
- FB101: footprint Capacitor_SMD:C_0805_2012Metric -> Capacitor_SMD:C_0805_2012Metric_Pad1.15x1.40mm_HandSolder
- moved C101 7.83 mm to (32.8, 50.5), turned to 180 degrees
- moved C102 5.87 mm to (42.7, 46.5), turned to 270 degrees
- renumbered J3 to J1, J4 to J102
Connections:
- MOD1 pad 1: GND -> Net-(J104-Pad2)
- MOD1 pad 2: +3V3 -> Net-(J103-Pad2)
Routing:
- net GND: track 85.1 -> 79.7 mm, vias 25 -> 26
- net +3V3: track 158.1 -> 153.5 mm, vias 5 -> 4
- net Net-(J104-Pad2): track 0.00 -> 3.70 mm
- net Net-(J103-Pad2): track 0.00 -> 2.72 mm
- net +5V: track 124.4 -> 122.0 mm

Commit message: Finished final changes and exported gerbers
Finished final changes and exported gerbers
Parts:
- moved R102 14.0 mm to (53.3, 63.9), turned to 90 degrees
- moved J103 2.00 mm to (60.2, 34.3)
- moved J104 2.00 mm to (55.6, 34.3)
- moved L1 1.71 mm to (47.2, 61.0), turned to 270 degrees
- moved R106 1.20 mm to (75.6, 70.6)
- moved R107 0.89 mm to (71.7, 71.3), turned to 180 degrees
- moved C4 0.60 mm to (71.5, 61.3)
- moved R111 0.52 mm to (64.0, 53.0)
- moved D2 0.35 mm to (40.3, 70.9)
Routing:
- net Net-(L1-Pad1): track 32.3 -> 15.6 mm
- net Net-(R102-Pad1): track 17.6 -> 3.74 mm
- net Net-(D2-Pad2): track 23.5 -> 20.0 mm
- net /V_boost_ctrl: track 49.8 -> 46.3 mm
- net /SWDIO: track 53.8 -> 56.5 mm, vias 0 -> 1
- net Net-(J103-Pad2): track 2.72 -> 4.09 mm
- net Net-(J104-Pad2): track 3.70 -> 2.46 mm
- net Net-(R106-Pad2): track 15.1 -> 16.3 mm
- net /SWCLK: track 33.9 -> 33.1 mm, vias 0 -> 1
- net GND: track 79.7 -> 79.0 mm
- net /SCK: track 15.8 -> 16.4 mm
- net +5V: track 122.0 -> 121.3 mm
- net +3V3: track 153.5 -> 154.1 mm, vias 4 -> 2
- net /Boost_out: vias 1 -> 0

Commit message: Added fiducials for automated assembly
Added fiducials for automated assembly
Parts:
- added TP10: Fiducial, Fiducial:Fiducial_0.75mm_Dia_1.5mm_Outer, F.Cu at (83.2, 83.6)
- added TP8: Fiducial, Fiducial:Fiducial_0.75mm_Dia_1.5mm_Outer, F.Cu at (87.7, 36.6)
- added TP9: Fiducial, Fiducial:Fiducial_0.75mm_Dia_1.5mm_Outer, F.Cu at (32.7, 79.8)
Changed lines of the file:
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@@
     (tracks 581)
     (zones 0)
-    (modules 76)
+    (modules 79)
     (nets 66)
   )
@@
     (visible_elements FFFFFF7F)
     (pcbplotparams
-      (layerselection 0x010fc_ffffffff)
+      (layerselection 0x010f8_ffffffff)
       (usegerberextensions false)
       (usegerberattributes false)
@@
     (add_net "Net-(U103-Pad46)")
   )
+  (module Fiducial:Fiducial_0.75mm_Dia_1.5mm_Outer (layer F.Cu)
+    (at 32.7 79.8)
+    (descr "Circular Fiducial, 0.75mm bare copper top; 1.5mm keepout (Level B)")
+    (tags marker)
+    (attr virtual)
+    (fp_text reference TP9 (at 0 -2) (layer F.SilkS)
+      (effects (font (size 1 1) (thickness 0.15)))
+    )
+    (fp_text value Fiducial (at 0 2) (layer F.Fab)
+      (effects (font (size 1 1) (thickness 0.15)))
+    )
+    (fp_circle (center 0 0) (end 0.75 0) (layer F.Fab) (width 0.1))
+    (fp_text user %R (at 0 0) (layer F.Fab)
+      (effects (font (size 0.3 0.3) (thickness 0.05)))
+    )
+    (fp_circle (center 0 0) (end 1 0) (layer F.CrtYd) (width 0.05))
+    (pad ~ smd circle (at 0 0) (size 0.75 0.75) (layers F.Cu F.Mask)
+      (solder_mask_margin 0.375) (clearance 0.375))
+  )
+  (module Fiducial:Fiducial_0.75mm_Dia_1.5mm_Outer (layer F.Cu)
+    (at 87.7 36.6)
+    (descr "Circular Fiducial, 0.75mm bare copper top; 1.5mm keepout (Level B)")
+    (tags marker)
+    (attr virtual)
+    (fp_text reference TP8 (at 0 2.1) (layer F.SilkS)
+      (effects (font (size 1 1) (thickness 0.15)))
+    )
+    (fp_text value Fiducial (at 0 2) (layer F.Fab)
+      (effects (font (size 1 1) (thickness 0.15)))
+    )
+    (fp_circle (center 0 0) (end 1 0) (layer F.CrtYd) (width 0.05))
+    (fp_text user %R (at 0 0) (layer F.Fab)
+      (effects (font (size 0.3 0.3) (thickness 0.05)))
+    )
+    (fp_circle (center 0 0) (end 0.75 0) (layer F.Fab) (width 0.1))
+    (pad ~ smd circle (at 0 0) (size 0.75 0.75) (layers F.Cu F.Mask)
+      (solder_mask_margin 0.375) (clearance 0.375))
+  )
+  (module Fiducial:Fiducial_0.75mm_Dia_1.5mm_Outer (layer F.Cu)
+    (at 83.2 83.6)
+    (descr "Circular Fiducial, 0.75mm bare copper top; 1.5mm keepout (Level B)")
+    (tags marker)
+    (attr virtual)
+    (fp_text reference TP10 (at 3 0.1) (layer F.SilkS)
+      (effects (font (size 1 1) (thickness 0.15)))
+    )
+    (fp_text value Fiducial (at 0 2) (layer F.Fab)
+      (effects (font (size 1 1) (thickness 0.15)))
+    )
+    (fp_circle (center 0 0) (end 0.75 0) (layer F.Fab) (width 0.1))
+    (fp_text user %R (at 0 0) (layer F.Fab)
+      (effects (font (size 0.3 0.3) (thickness 0.05)))
+    )
+    (fp_circle (center 0 0) (end 1 0) (layer F.CrtYd) (width 0.05))
+    (pad ~ smd circle (at 0 0) (size 0.75 0.75) (layers F.Cu F.Mask)
+      (solder_mask_margin 0.375) (clearance 0.375))
+  )
   (module powersupply:Default_Jumper (layer B.Cu)

Commit message: changes
Parts:
- moved TP9 3.45 mm to (34.0, 83.0)
- moved TP8 0.92 mm to (87.0, 36.0)
- moved TP10 0.63 mm to (83.0, 83.0)
- moved TP4 0.34 mm to (75.5, 57.0)
Changed lines of the file:
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@@
-(kicad_pcb (version 20171130) (host pcbnew "(5.0.1-3-g963ef8bb5)")
+(kicad_pcb (version 20171130) (host pcbnew "(5.1.4-0-10_14)")
   (general
     (thickness 1.6)
-    (drawings 28)
+    (drawings 20)
     (tracks 581)
     (zones 0)
@@
     (zone_45_only no)
     (trace_min 0.2)
-    (segment_width 0.2)
-    (edge_width 0.05)
     (via_size 0.8)
     (via_drill 0.4)
@@
     (uvia_min_size 0.2)
     (uvia_min_drill 0.1)
+    (edge_width 0.05)
+    (segment_width 0.2)
     (pcb_text_width 0.3)
     (pcb_text_size 1.5 1.5)
@@
   )
   (module Fiducial:Fiducial_0.75mm_Dia_1.5mm_Outer (layer F.Cu)
-    (at 32.7 79.8)
+    (at 34 83)
     (descr "Circular Fiducial, 0.75mm bare copper top; 1.5mm keepout (Level B)")
     (tags marker)
@@
   )
   (module Fiducial:Fiducial_0.75mm_Dia_1.5mm_Outer (layer F.Cu)
-    (at 87.7 36.6)
+    (at 87 36)
     (descr "Circular Fiducial, 0.75mm bare copper top; 1.5mm keepout (Level B)")
     (tags marker)
     (attr virtual)
-    (fp_text reference TP8 (at 0 2.1) (layer F.SilkS)
+    (fp_text reference TP8 (at 0.8 2.15) (layer F.SilkS)
       (effects (font (size 1 1) (thickness 0.15)))
     )
@@
   )
   (module Fiducial:Fiducial_0.75mm_Dia_1.5mm_Outer (layer F.Cu)
-    (at 83.2 83.6)
+    (at 83 83)
     (descr "Circular Fiducial, 0.75mm bare copper top; 1.5mm keepout (Level B)")
     (tags marker)
@@
   )
   (module Connector_PinHeader_2.54mm:PinHeader_1x01_P2.54mm_Vertical (layer F.Cu)
-    (at 75.8 56.9)
+    (at 75.5 57.05)
     (descr "Through hole straight pin header, 1x01, 2.54mm pitch, single row")
     (tags "Through hole pin header THT 1x01 2.54mm single row")
@@
   (gr_arc (start 86.12 31.55) (end 89.57 31.55) (angle -90) (layer Edge.Cuts) (width 0.05))
   (gr_arc (start 32.27 87.95) (end 28.82 87.95) (angle -89.66785427) (layer Edge.Cuts) (width 0.05))
-  (gr_line (start 59.15 34.58) (end 59.15 35) (layer B.SilkS) (width 0.12))
-  (gr_line (start 59.15 35.3) (end 59.15 35.72) (layer B.SilkS) (width 0.12))
-  (gr_line (start 59.15 33.15) (end 59.15 33.57) (layer B.SilkS) (width 0.12))
-  (gr_line (start 59.15 33.88) (end 59.15 34.3) (layer B.SilkS) (width 0.12))
-  (gr_line (start 55.91 35.29) (end 55.91 35.71) (layer B.SilkS) (width 0.12))
-  (gr_line (start 55.91 34.57) (end 55.91 34.99) (layer B.SilkS) (width 0.12))
-  (gr_line (start 55.91 33.87) (end 55.91 34.29) (layer B.SilkS) (width 0.12))
-  (gr_line (start 55.91 33.14) (end 55.91 33.56) (layer B.SilkS) (width 0.12))
-  (gr_text "Variable\nPower Supply" (at 59.32 43.15) (layer B.SilkS)
-    (effects (font (size 5 5) (thickness 1)) (justify mirror))
+  (gr_text "Variable\nPower Supply" (at 59.2 46.35) (layer B.SilkS)
+    (effects (font (size 2.5 2.5) (thickness 0.625)) (justify mirror))
   )
   (gr_arc (start 32.27 31.55) (end 32.27 28.1) (angle -90) (layer Edge.Cuts) (width 0.05))
